Commit message: wheels are not shown yet

File: urdf/barista_robot_model.urdf (robot description, URDF)
Before this commit: robot barista_bot, 10 links, 9 joints
Links:
- removed link back_pitch_link
- removed link back_roll_link
- removed link back_yaw_link
- removed link front_pitch_link
- removed link front_roll_link
- removed link front_yaw_link
- removed link main body
- removed link right_wheel
- added link main_body; visual cylinder length=0.155 radius=0.1825
Joints:
- removed joint back_pitch_joint
- removed joint back_roll_joint
- removed joint back_yaw_joint
- removed joint base_link_joint
- removed joint front_pitch_joint
- removed joint front_roll_joint
- removed joint front_yaw_joint
- removed joint joint_right_wheel
- added joint base_body_joint: type fixed, parent base_link, child main_body, origin xyz=0 0 .1127 rpy=0 0 0
- joint joint_left_wheel: origin xyz=0 0.05 -0.025 rpy=0 0 0 -> xyz=0 0.150 -0.0352 rpy=0 0 0; parent chassis -> main_body

Commit message: main body, wheels, caster wheels and laser are added

File: urdf/barista_robot_model.urdf (robot description, URDF)
Before this commit: robot barista_bot, 3 links, 2 joints
Links:
- removed link main_body
- added link back_caster, mass 0.5; collision sphere radius=0.0352; visual sphere radius=0.0352
- added link base_footprint
- added link front_caster, mass 0.5; collision sphere radius=0.0352; visual sphere radius=0.0352
- added link front_laser, mass 0.05; collision cylinder length=0.02 radius=0.025; visual cylinder length=0.02 radius=0.025
- added link right_wheel, mass 1.5; collision cylinder length=0.05 radius=0.025; visual cylinder length=0.0206 radius=0.0352
- link base_link: mass None -> 20.5; geometry collision cylinder length=0.155 radius=0.178; visual cylinder length=0.155 radius=0.178
- link left_wheel: mass None -> 1.5; geometry collision cylinder length=0.05 radius=0.025; visual cylinder length=0.0206 radius=0.0352
Joints:
- removed joint base_body_joint
- removed joint joint_left_wheel
- added joint base_joint: type fixed, parent base_footprint, child base_link, origin xyz=0 0 0.1127
- added joint front_caster_wheel_joint: type fixed, parent base_link, child front_caster, origin xyz=0.1 0.0 -0.0775 rpy=0 0 0, axis 0 0 0
- added joint front_laser_joint: type fixed, parent base_link, child front_laser, origin xyz=0.14 0.0 0.0875 rpy=-3.14 0 0, axis 0 0 0
- added joint left_wheel_joint: type continuous, parent base_link, child left_wheel, origin xyz=0 0.15 -0.0775 rpy=-1.57 0 0, axis 0 0 1
- added joint rear_caster_wheel_joint: type fixed, parent base_link, child back_caster, origin xyz=-0.1 0.0 -0.0775 rpy=0 0 0, axis 0 0 0
- added joint right_wheel_joint: type continuous, parent base_link, child right_wheel, origin xyz=0 -0.15 -0.0775 rpy=1.57 0 0, axis 0 0 -1

Commit message: added top tray

File: urdf/barista_robot_model.urdf (robot description, URDF)
Before this commit: robot barista_bot, 7 links, 6 joints
Links:
- added link Cup_Holder_Tray_link, mass 20.5; collision cylinder length=0.090 radius=0.160; visual cylinder length=0.090 radius=0.160
Joints:
- added joint Cup_Holder_Tray_Joint: type fixed, parent base_link, child Cup_Holder_Tray_link, origin xyz=0 0 0.3425

Commit message: added one of stands

File: urdf/barista_robot_model.urdf (robot description, URDF)
Before this commit: robot barista_bot, 8 links, 7 joints
Links:
- added link Standoff_Rod_1_link, mass 0.5; collision cylinder length=0.22 radius=0.01; visual cylinder length=0.22 radius=0.01
Joints:
- added joint Standoff_Rod_1_Joint: type fixed, parent base_link, child Standoff_Rod_1_link, origin xyz=0.1 0.1 0.1875

Commit message: added laser STL

File: urdf/barista_robot_model.urdf (robot description, URDF)
Before this commit: robot barista_bot, 9 links, 8 joints
Links:
- link front_laser: geometry collision cylinder length=0.02 radius=0.025; visual mesh filename=package://barista_robot_description/meshes/lidar_m10_p.STL scale=1 1 1
Joints:
- joint front_laser_joint: origin xyz=0.14 0.0 0.0875 rpy=-3.14 0 0 -> xyz=0.14 0.0 0.0775 rpy=0 0 0

Commit message: added 4 poles

File: urdf/barista_robot_model.urdf (robot description, URDF)
Before this commit: robot barista_bot, 9 links, 8 joints
Links:
- added link Standoff_Rod_2_link, mass 0.5; collision cylinder length=0.22 radius=0.01; visual cylinder length=0.22 radius=0.01
- added link Standoff_Rod_3_link, mass 0.5; collision cylinder length=0.22 radius=0.01; visual cylinder length=0.22 radius=0.01
- added link Standoff_Rod_4_link, mass 0.5; collision cylinder length=0.22 radius=0.01; visual cylinder length=0.22 radius=0.01
Joints:
- added joint Standoff_Rod_2_Joint: type fixed, parent base_link, child Standoff_Rod_2_link, origin xyz=-0.1 -0.1 0.1875
- added joint Standoff_Rod_3_Joint: type fixed, parent base_link, child Standoff_Rod_3_link, origin xyz=0.1 -0.1 0.1875
- added joint Standoff_Rod_4_Joint: type fixed, parent base_link, child Standoff_Rod_4_link, origin xyz=-0.1 0.1 0.1875

Commit message: now working

File: urdf/barista_robot_model.urdf (robot description, URDF)
Before this commit: robot barista_bot, 12 links, 11 joints
Links:
- link Cup_Holder_Tray_link: mass 20.5 -> 10.0
- link base_link: mass 20.5 -> 10.0
- link front_laser: geometry collision cylinder length=0.02 radius=0.025; visual cylinder length=0.02 radius=0.025
- link left_wheel: geometry collision cylinder length=0.0206 radius=0.0352; visual cylinder length=0.0206 radius=0.0352
- link right_wheel: geometry collision cylinder length=0.0206 radius=0.0352; visual cylinder length=0.0206 radius=0.0352
Joints:
- joint front_laser_joint: origin xyz=0.14 0.0 0.0775 rpy=0 0 0 -> xyz=0.14 0.0 0.0875 rpy=0 0 0

Commit message: color updated.

File: urdf/barista_robot_model.urdf (robot description, URDF)
Before this commit: robot barista_bot, 12 links, 11 joints
Links:
- link Cup_Holder_Tray_link: mass 10.0 -> 8.0
- link front_laser: geometry collision cylinder length=0.02 radius=0.025; visual mesh filename=package://barista_robot_description/meshes/lidar_m10_p.STL scale=1 1 1

Commit message: launch joint state publisher from urdf

File: urdf/barista_robot_model.urdf (robot description, URDF)
Before this commit: robot barista_bot, 12 links, 11 joints
Joints:
- joint front_laser_joint: origin xyz=0.14 0.0 0.0875 rpy=0 0 0 -> xyz=0.14 0.0 0.0775 rpy=0 0 0

Commit message: Laser lay visulization is not stable but others works well

File: urdf/barista_robot_model.urdf (robot description, URDF)
Before this commit: robot barista_bot, 12 links, 11 joints
Links:
- link front_laser: geometry collision cylinder length=0.02 radius=0.025; visual cylinder length=0.02 radius=0.025
Joints:
- joint front_laser_joint: origin xyz=0.14 0.0 0.0775 rpy=0 0 0 -> xyz=0.14 0.0 0.0875 rpy=0 0 0

Commit message: created xacro files

File: urdf/barista_robot_model.urdf (robot description, URDF)
Before this commit: robot barista_bot, 12 links, 11 joints
Links:
- link front_laser: geometry collision cylinder length=0.06 radius=0.025; visual mesh filename=package://barista_robot_description/meshes/sick_s3000.dae scale=0.2 0.2 0.2
Joints:
- joint front_laser_joint: axis 0 0 0 -> (none); origin xyz=0.14 0.0 0.0875 rpy=0 0 0 -> xyz=0.14 0.0 0.0775 rpy=0 0 0

Commit message: make some change in task1

File: urdf/barista_robot_model.urdf (robot description, URDF)
Before this commit: robot barista_bot, 12 links, 11 joints
Links:
- link front_laser: geometry collision cylinder length=0.02 radius=0.025; visual mesh filename=package://barista_robot_description/meshes/sick_s3000.dae scale=0.2 0.2 0.2
Joints:
- joint front_laser_joint: origin xyz=0.14 0.0 0.0875 rpy=0 0 0 -> xyz=0.14 0.0 0.0775 rpy=0 0 0

Commit message: laser position changed

File: urdf/barista_robot_model.urdf (robot description, URDF)
Before this commit: robot barista_bot, 12 links, 11 joints
Joints:
- joint front_laser_joint: origin xyz=0.14 0.0 0.0775 rpy=0 0 0 -> xyz=0.14 0.0 0.078 rpy=0 0 0

Commit message: Updated code for task1

File: urdf/barista_robot_model.urdf (robot description, URDF)
Before this commit: robot barista_bot, 12 links, 11 joints
Joints:
- joint Standoff_Rod_1_Joint: origin xyz=0.1 0.1 0.1875 -> xyz=0.05 0.14 0.1875
- joint Standoff_Rod_2_Joint: origin xyz=-0.1 -0.1 0.1875 -> xyz=-0.05 -0.14 0.1875
- joint Standoff_Rod_3_Joint: origin xyz=0.1 -0.1 0.1875 -> xyz=0.05 -0.14 0.1875
- joint Standoff_Rod_4_Joint: origin xyz=-0.1 0.1 0.1875 -> xyz=-0.05 0.14 0.1875

Commit message: Final revisions for task2

File: urdf/barista_robot_model.urdf (robot description, URDF)
Before this commit: robot barista_bot, 12 links, 11 joints
Joints:
- joint Standoff_Rod_1_Joint: origin xyz=0.1 0.1 0.1875 -> xyz=0.05 0.14 0.1875
- joint Standoff_Rod_2_Joint: origin xyz=-0.1 -0.1 0.1875 -> xyz=-0.05 -0.14 0.1875
- joint Standoff_Rod_3_Joint: origin xyz=0.1 -0.1 0.1875 -> xyz=0.05 -0.14 0.1875
- joint Standoff_Rod_4_Joint: origin xyz=-0.1 0.1 0.1875 -> xyz=-0.05 0.14 0.1875

File: xacro/standoff_rod.xacro (robot description, xacro)
@@ -5,5 +5,5 @@
         <parent link="base_link"/>
         <child link="Standoff_Rod_1_link"/>
-        <origin xyz="0.1 0.1 0.1875"/>
+        <origin xyz="0.05 0.14 0.1875"/>
     </joint>
     <link name="Standoff_Rod_1_link">
@@ -31,5 +31,5 @@
         <parent link="base_link"/>
         <child link="Standoff_Rod_2_link"/>
-        <origin xyz="-0.1 -0.1 0.1875"/>
+        <origin xyz="-0.05 -0.14 0.1875"/>
     </joint>
     <link name="Standoff_Rod_2_link">
@@ -57,5 +57,5 @@
         <parent link="base_link"/>
         <child link="Standoff_Rod_3_link"/>
-        <origin xyz="0.1 -0.1 0.1875"/>
+        <origin xyz="0.05 -0.14 0.1875"/>
     </joint>
     <link name="Standoff_Rod_3_link">
@@ -83,5 +83,5 @@
         <parent link="base_link"/>
         <child link="Standoff_Rod_4_link"/>
-        <origin xyz="-0.1 0.1 0.1875"/>
+        <origin xyz="-0.05 0.14 0.1875"/>
     </joint>
     <link name="Standoff_Rod_4_link">
