Commit message: converting to instructed format, not working

File: xacro/barista_robot_model.urdf.xacro (robot description, xacro)
@@ -1,15 +1,15 @@
-<!-- barista_robot_model.urdf.xacro -->
-<xacro:robot xmlns:xacro="http://ros.org/wiki/xacro" name="barista_bot">
+<?xml version="1.0"?>
+<robot xmlns:xacro="http://www.ros.org/wiki/xacro" name="barista_bot">
   <!-- Load Material Colors -->
-  <xacro:include filename="${file_path}/materials.xacro" />
+  <xacro:include filename="$(find barista_robot_description)/xacro/materials.xacro" />
   <!-- Properties -->
   <xacro:property name="wheel_radius" value="0.0352"/>
   <xacro:property name="wheel_width" value="0.0206"/>
   <!-- Include Macro Files -->
-  <xacro:include filename="${file_path}/drive_wheel.xacro"/>
-  <xacro:include filename="${file_path}/caster_wheel.xacro"/>
-  <xacro:include filename="${file_path}/standoff_rod.xacro"/>
-  <xacro:include filename="${file_path}/cup_holder_tray.xacro"/>
-  <xacro:include filename="${file_path}/laser_scanner.xacro"/>
+  <xacro:include filename="$(find barista_robot_description)/xacro/drive_wheel.xacro"/>
+  <xacro:include filename="$(find barista_robot_description)/xacro/caster_wheel.xacro"/>
+  <xacro:include filename="$(find barista_robot_description)/xacro/standoff_rod.xacro"/>
+  <xacro:include filename="$(find barista_robot_description)/xacro/cup_holder_tray.xacro"/>
+  <xacro:include filename="$(find barista_robot_description)/xacro/laser_scanner.xacro"/>
   <!-- Base Footprint -->
   <link name="base_footprint"/>
@@ -56,3 +56,3 @@
     <xacro:laser_scanner parent="base_link" xyz="0.14 0.0 0.0775"/>
   </xacro:if>
-</xacro:robot>
+</robot>

File: xacro/caster_wheel.xacro (robot description, xacro)
@@ -1,3 +1,4 @@
-<xacro:macro name="caster_wheel" params="name parent xyz">
+<?xml version="1.0"?>
+<robot xmlns:xacro="http://www.ros.org/wiki/xacro" name="caster_wheel" params="name parent xyz">
   <joint name="${name}_joint" type="fixed">
     <parent link="${parent}"/>
@@ -30,3 +31,3 @@
     <material>Gazebo/Gray</material>
   </gazebo>
-</xacro:macro>
+</robot>

File: xacro/cup_holder_tray.xacro (robot description, xacro)
@@ -1,3 +1,4 @@
-<xacro:macro name="cup_holder_tray" params="parent xyz">
+<?xml version="1.0"?>
+<robot xmlns:xacro="http://www.ros.org/wiki/xacro" name="cup_holder_tray" params="parent xyz">
   <joint name="Cup_Holder_Tray_Joint" type="fixed">
     <parent link="${parent}"/>
@@ -26,3 +27,3 @@
     <material>Gazebo/Blue</material>
   </gazebo>
-</xacro:macro>
+</robot>

File: xacro/drive_wheel.xacro (robot description, xacro)
@@ -1,3 +1,4 @@
-<xacro:macro name="drive_wheel" params="side parent xyz rpy axis">
+<?xml version="1.0"?>
+<robot xmlns:xacro="http://www.ros.org/wiki/xacro" name="drive_wheel" params="side parent xyz rpy axis">
   <joint name="${side}_wheel_joint" type="continuous">
     <parent link="${parent}"/>
@@ -32,3 +33,3 @@
     <material>Gazebo/Black</material>
   </gazebo>
-</xacro:macro>
+</robot>

File: xacro/laser_scanner.xacro (robot description, xacro)
@@ -1,3 +1,4 @@
-<xacro:macro name="laser_scanner" params="parent xyz">
+<?xml version="1.0"?>
+<robot xmlns:xacro="http://www.ros.org/wiki/xacro" name="laser_scanner" params="parent xyz">
   <joint name="front_laser_joint" type="fixed">
     <parent link="${parent}"/>
@@ -49,3 +50,3 @@
     </sensor>
   </gazebo>
-</xacro:macro>
+</robot>

File: xacro/materials.xacro (robot description, xacro)
@@ -16,3 +16,3 @@
     <color rgba="1 0 0 1"/>
   </material>
-</xacro:macro>
+</robot>

File: xacro/standoff_rod.xacro (robot description, xacro)
@@ -1,3 +1,4 @@
-<xacro:macro name="standoff_rod" params="name parent xyz">
+<?xml version="1.0"?>
+<robot xmlns:xacro="http://www.ros.org/wiki/xacro" name="standoff_rod" params="name parent xyz">
   <joint name="${name}_Joint" type="fixed">
     <parent link="${parent}"/>
@@ -26,3 +27,3 @@
     <material>Gazebo/white</material>
   </gazebo>
-</xacro:macro>
+</robot>

Commit message: it works.. laser issue argument issue

File: xacro/barista_robot_model.urdf.xacro (robot description, xacro)
@@ -1,9 +1,7 @@
 <?xml version="1.0"?>
 <robot xmlns:xacro="http://www.ros.org/wiki/xacro" name="barista_bot">
+  <xacro:arg name="include_laser" default="true"/>
   <!-- Load Material Colors -->
-  <xacro:include filename="$(find barista_robot_description)/xacro/materials.xacro" />
-  <!-- Properties -->
-  <xacro:property name="wheel_radius" value="0.0352"/>
-  <xacro:property name="wheel_width" value="0.0206"/>
+  <xacro:include filename="$(find barista_robot_description)/xacro/materials.xacro"/>
   <!-- Include Macro Files -->
   <xacro:include filename="$(find barista_robot_description)/xacro/drive_wheel.xacro"/>
@@ -12,5 +10,5 @@
   <xacro:include filename="$(find barista_robot_description)/xacro/cup_holder_tray.xacro"/>
   <xacro:include filename="$(find barista_robot_description)/xacro/laser_scanner.xacro"/>
-  <!-- Base Footprint -->
+  <!-- Base -->
   <link name="base_footprint"/>
   <joint name="base_joint" type="fixed">
@@ -19,40 +17,26 @@
     <origin xyz="0 0 0.1127"/>
   </joint>
-  <!-- Base Link -->
   <link name="base_link">
-    <inertial>
-      <mass value="10.0"/>
-      <origin xyz="0 0 0"/>
-      <inertia ixx="0.0992" ixy="0.0" ixz="0.0" iyy="0.0992" iyz="0.0" izz="0.1584"/>
-    </inertial>
-    <visual>
-      <geometry>
-        <cylinder radius="0.178" length="0.155"/>
-      </geometry>
-      <material name="blue"/>
-    </visual>
-    <collision>
-      <geometry>
-        <cylinder radius="0.178" length="0.155"/>
-      </geometry>
-    </collision>
+    <visual><geometry><cylinder radius="0.178" length="0.155"/></geometry></visual>
+    <collision><geometry><cylinder radius="0.178" length="0.155"/></geometry></collision>
+    <inertial><mass value="10.0"/></inertial>
   </link>
-  <!-- Drive Wheels -->
+  <!-- Wheels -->
   <xacro:drive_wheel side="left" parent="base_link" xyz="0 0.15 -0.0775" rpy="-1.57 0 0" axis="0 0 1"/>
   <xacro:drive_wheel side="right" parent="base_link" xyz="0 -0.15 -0.0775" rpy="1.57 0 0" axis="0 0 -1"/>
-  <!-- Caster Wheels -->
+  <!-- Casters -->
   <xacro:caster_wheel name="front_caster" parent="base_link" xyz="0.1 0.0 -0.0775"/>
   <xacro:caster_wheel name="back_caster" parent="base_link" xyz="-0.1 0.0 -0.0775"/>
-  <!-- Standoff Rods -->
+  <!-- Standoffs -->
   <xacro:standoff_rod name="Standoff_Rod_1" parent="base_link" xyz="0.1 0.1 0.1875"/>
   <xacro:standoff_rod name="Standoff_Rod_2" parent="base_link" xyz="-0.1 -0.1 0.1875"/>
   <xacro:standoff_rod name="Standoff_Rod_3" parent="base_link" xyz="0.1 -0.1 0.1875"/>
   <xacro:standoff_rod name="Standoff_Rod_4" parent="base_link" xyz="-0.1 0.1 0.1875"/>
-  <!-- Cup Holder Tray -->
+  <!-- Tray -->
   <xacro:cup_holder_tray parent="base_link" xyz="0 0 0.3425"/>
-  <!-- Laser Scanner with conditional argument -->
-  <xacro:arg name="include_laser" default="true"/>
-  <xacro:if value="${include_laser}">
+  <!-- Optional laser -->
+  <!-- <xacro:if value="${include_laser}">
     <xacro:laser_scanner parent="base_link" xyz="0.14 0.0 0.0775"/>
-  </xacro:if>
+  </xacro:if> -->
+  <xacro:laser_scanner parent="base_link" xyz="0.14 0.0 0.0775"/>
 </robot>

File: xacro/caster_wheel.xacro (robot description, xacro)
@@ -1,33 +1,15 @@
 <?xml version="1.0"?>
-<robot xmlns:xacro="http://www.ros.org/wiki/xacro" name="caster_wheel" params="name parent xyz">
-  <joint name="${name}_joint" type="fixed">
-    <parent link="${parent}"/>
-    <child link="${name}"/>
-    <origin xyz="${xyz}" rpy="0 0 0"/>
-  </joint>
-  <link name="${name}">
-    <visual>
-      <geometry>
-        <sphere radius="0.0352"/>
-      </geometry>
-    </visual>
-    <collision>
-      <geometry>
-        <sphere radius="0.0352"/>
-      </geometry>
-    </collision>
-    <inertial>
-      <mass value="0.5"/>
-      <origin xyz="0 0 0" rpy="0 0 0"/>
-      <inertia ixx="9.479166666666669e-06" ixy="0.0" ixz="0.0" iyy="9.479166666666669e-06" iyz="0.0" izz="1.5625000000000004e-05"/>
-    </inertial>
-  </link>
-  <gazebo reference="${name}">
-    <mu1 value="0.0"/>
-    <mu2 value="0.0"/>
-    <kp value="10000000.0"/>
-    <kd value="100.0"/>
-    <fdir1 value="0 0 1"/>
-    <material>Gazebo/Gray</material>
-  </gazebo>
+<robot xmlns:xacro="http://www.ros.org/wiki/xacro" name="barista_bot">
+  <xacro:macro name="caster_wheel" params="name parent xyz">
+    <joint name="${name}_joint" type="fixed">
+      <parent link="${parent}"/>
+      <child link="${name}"/>
+      <origin xyz="${xyz}"/>
+    </joint>
+    <link name="${name}">
+      <visual><geometry><sphere radius="0.0352"/></geometry></visual>
+      <collision><geometry><sphere radius="0.0352"/></geometry></collision>
+      <inertial><mass value="0.5"/></inertial>
+    </link>
+  </xacro:macro>
 </robot>

File: xacro/cup_holder_tray.xacro (robot description, xacro)
@@ -1,29 +1,15 @@
 <?xml version="1.0"?>
-<robot xmlns:xacro="http://www.ros.org/wiki/xacro" name="cup_holder_tray" params="parent xyz">
-  <joint name="Cup_Holder_Tray_Joint" type="fixed">
-    <parent link="${parent}"/>
-    <child link="Cup_Holder_Tray_link"/>
-    <origin xyz="${xyz}"/>
-  </joint>
-  <link name="Cup_Holder_Tray_link">
-    <inertial>
-      <mass value="8.0"/>
-      <origin xyz="0 0 0" rpy="0 0 0"/>
-      <inertia ixx="0.0566" ixy="0.0" ixz="0.0" iyy="0.0566" iyz="0.0" izz="0.1024"/>
-    </inertial>
-    <visual>
-      <geometry>
-        <cylinder radius="0.160" length="0.090"/>
-      </geometry>
-      <material name="blue"/>
-    </visual>
-    <collision>
-      <geometry>
-        <cylinder radius="0.160" length="0.090"/>
-      </geometry>
-    </collision>
-  </link>
-  <gazebo reference="Cup_Holder_Tray_link">
-    <material>Gazebo/Blue</material>
-  </gazebo>
+<robot xmlns:xacro="http://www.ros.org/wiki/xacro" name="barista_bot">
+  <xacro:macro name="cup_holder_tray" params="parent xyz">
+    <joint name="Cup_Holder_Tray_Joint" type="fixed">
+      <parent link="${parent}"/>
+      <child link="Cup_Holder_Tray_link"/>
+      <origin xyz="${xyz}"/>
+    </joint>
+    <link name="Cup_Holder_Tray_link">
+      <visual><geometry><cylinder radius="0.160" length="0.090"/></geometry></visual>
+      <collision><geometry><cylinder radius="0.160" length="0.090"/></geometry></collision>
+      <inertial><mass value="8.0"/></inertial>
+    </link>
+  </xacro:macro>
 </robot>

File: xacro/drive_wheel.xacro (robot description, xacro)
@@ -1,35 +1,16 @@
 <?xml version="1.0"?>
-<robot xmlns:xacro="http://www.ros.org/wiki/xacro" name="drive_wheel" params="side parent xyz rpy axis">
-  <joint name="${side}_wheel_joint" type="continuous">
-    <parent link="${parent}"/>
-    <child link="${side}_wheel"/>
-    <origin xyz="${xyz}" rpy="${rpy}"/>
-    <axis xyz="${axis}"/>
-  </joint>
-  <link name="${side}_wheel">
-    <inertial>
-      <mass value="1.5"/>
-      <origin xyz="0 0 0" rpy="0 0 0"/>
-      <inertia ixx="0.000517685" ixy="0.0" ixz="0.0" iyy="0.000517685" iyz="0.0" izz="0.00092928"/>
-    </inertial>
-    <visual>
-      <geometry>
-        <cylinder radius="${wheel_radius}" length="${wheel_width}"/>
-      </geometry>
-      <material name="black"/>
-    </visual>
-    <collision>
-      <geometry>
-        <cylinder radius="${wheel_radius}" length="${wheel_width}"/>
-      </geometry>
-    </collision>
-  </link>
-  <gazebo reference="${side}_wheel">
-    <mu1 value="1.0"/>
-    <mu2 value="0.8"/>
-    <kp value="1000000.0"/>
-    <kd value="10.0"/>
-    <fdir1 value="1 0 0"/>
-    <material>Gazebo/Black</material>
-  </gazebo>
+<robot xmlns:xacro="http://www.ros.org/wiki/xacro" name="barista_bot">
+  <xacro:macro name="drive_wheel" params="side parent xyz rpy axis">
+    <joint name="${side}_wheel_joint" type="continuous">
+      <parent link="${parent}"/>
+      <child link="${side}_wheel"/>
+      <origin xyz="${xyz}" rpy="${rpy}"/>
+      <axis xyz="${axis}"/>
+    </joint>
+    <link name="${side}_wheel">
+      <visual><geometry><cylinder radius="0.0352" length="0.0206"/></geometry></visual>
+      <collision><geometry><cylinder radius="0.0352" length="0.0206"/></geometry></collision>
+      <inertial><mass value="1.5"/></inertial>
+    </link>
+  </xacro:macro>
 </robot>

File: xacro/laser_scanner.xacro (robot description, xacro)
@@ -1,52 +1,15 @@
 <?xml version="1.0"?>
-<robot xmlns:xacro="http://www.ros.org/wiki/xacro" name="laser_scanner" params="parent xyz">
-  <joint name="front_laser_joint" type="fixed">
-    <parent link="${parent}"/>
-    <child link="front_laser"/>
-    <origin xyz="${xyz}" rpy="0 0 0"/>
-  </joint>
-  <link name="front_laser">
-    <inertial>
-      <mass value="0.05"/>
-      <origin xyz="0 0 0" rpy="0 0 0"/>
-      <inertia ixx="0.000252666667" ixy="0" ixz="0" iyy="0.000252666667" iyz="0" izz="0.0005"/>
-    </inertial>
-    <visual>
-      <geometry>
-        <mesh filename=\"package://barista_robot_description/meshes/sick_s3000.dae\" scale=\"0.2 0.2 0.2\"/>
-      </geometry>
-      <material name=\"red\"/>
-    </visual>
-    <collision>
-      <geometry>
-        <cylinder radius=\"0.025\" length=\"0.06\"/>
-      </geometry>
-    </collision>
-  </link>
-  <gazebo reference=\"front_laser\">
-    <sensor name=\"front_laser_ray\" type=\"ray\">
-      <pose>0.03 0 0.02 0 0 0</pose>
-      <ray>
-        <scan>
-          <horizontal>
-            <samples>200</samples>
-            <resolution>1.0</resolution>
-            <min_angle>-1.57</min_angle>
-            <max_angle>1.57</max_angle>
-          </horizontal>
-        </scan>
-        <range>
-          <min>0.1</min>
-          <max>5.0</max>
-        </range>
-      </ray>
-      <plugin name=\"laser\" filename=\"libgazebo_ros_ray_sensor.so\">
-        <ros><remapping>~/out:=scan</remapping></ros>
-        <output_type>sensor_msgs/LaserScan</output_type>
-      </plugin>
-      <visualize>true</visualize>
-      <update_rate>30.0</update_rate>
-      <always_on>true</always_on>
-    </sensor>
-  </gazebo>
+<robot xmlns:xacro="http://www.ros.org/wiki/xacro" name="barista_bot">
+  <xacro:macro name="laser_scanner" params="parent xyz">
+    <joint name="front_laser_joint" type="fixed">
+      <parent link="${parent}"/>
+      <child link="front_laser"/>
+      <origin xyz="${xyz}"/>
+    </joint>
+    <link name="front_laser">
+      <visual><geometry><cylinder radius="0.025" length="0.06"/></geometry></visual>
+      <collision><geometry><cylinder radius="0.025" length="0.06"/></geometry></collision>
+      <inertial><mass value="0.05"/></inertial>
+    </link>
+  </xacro:macro>
 </robot>

File: xacro/materials.xacro (robot description, xacro)
@@ -1,18 +1,7 @@
 <?xml version="1.0"?>
-<robot xmlns:xacro="http://www.ros.org/wiki/xacro" name="load_custom_materials" params="">
-  <material name="white">
-    <color rgba="1 1 1 1"/>
-  </material>
-  <material name="orange">
-    <color rgba="1 0.3 0.1 1"/>
-  </material>
-  <material name="blue">
-    <color rgba="0.2 0.2 1 1"/>
-  </material>
-  <material name="black">
-    <color rgba="0 0 0 1"/>
-  </material>
-  <material name="red">
-    <color rgba="1 0 0 1"/>
-  </material>
+<robot xmlns:xacro="http://www.ros.org/wiki/xacro" name="barista_bot">
+  <material name="white"><color rgba="1 1 1 1"/></material>
+  <material name="blue"><color rgba="0.2 0.2 1 1"/></material>
+  <material name="black"><color rgba="0 0 0 1"/></material>
+  <material name="red"><color rgba="1 0 0 1"/></material>
 </robot>

File: xacro/standoff_rod.xacro (robot description, xacro)
@@ -1,29 +1,15 @@
 <?xml version="1.0"?>
-<robot xmlns:xacro="http://www.ros.org/wiki/xacro" name="standoff_rod" params="name parent xyz">
-  <joint name="${name}_Joint" type="fixed">
-    <parent link="${parent}"/>
-    <child link="${name}_link"/>
-    <origin xyz="${xyz}"/>
-  </joint>
-  <link name="${name}_link">
-    <inertial>
-      <mass value="0.5"/>
-      <origin xyz="0 0 0" rpy="0 0 0"/>
-      <inertia ixx="0.0020291666666666665" ixy="0.0" ixz="0.0" iyy="0.0020291666666666665" iyz="0.0" izz="2.5e-05"/>
-    </inertial>
-    <visual>
-      <geometry>
-        <cylinder radius="0.01" length="0.22"/>
-      </geometry>
-      <material name="white"/>
-    </visual>
-    <collision>
-      <geometry>
-        <cylinder radius="0.01" length="0.22"/>
-      </geometry>
-    </collision>
-  </link>
-  <gazebo reference="${name}_link">
-    <material>Gazebo/white</material>
-  </gazebo>
+<robot xmlns:xacro="http://www.ros.org/wiki/xacro" name="barista_bot">
+  <xacro:macro name="standoff_rod" params="name parent xyz">
+    <joint name="${name}_Joint" type="fixed">
+      <parent link="${parent}"/>
+      <child link="${name}_link"/>
+      <origin xyz="${xyz}"/>
+    </joint>
+    <link name="${name}_link">
+      <visual><geometry><cylinder radius="0.01" length="0.22"/></geometry></visual>
+      <collision><geometry><cylinder radius="0.01" length="0.22"/></geometry></collision>
+      <inertial><mass value="0.5"/></inertial>
+    </link>
+  </xacro:macro>
 </robot>
