Commit message: using box bot platform and add more objects on it.

File: xacro/barista_robot_model.urdf.xacro (robot description, xacro)
@@ -1,42 +1,33 @@
 <?xml version="1.0"?>
 <robot xmlns:xacro="http://www.ros.org/wiki/xacro" name="barista_bot">
-  <xacro:arg name="include_laser" default="true"/>
-  <!-- Load Material Colors -->
-  <xacro:include filename="$(find barista_robot_description)/xacro/materials.xacro"/>
-  <!-- Include Macro Files -->
-  <xacro:include filename="$(find barista_robot_description)/xacro/drive_wheel.xacro"/>
-  <xacro:include filename="$(find barista_robot_description)/xacro/caster_wheel.xacro"/>
-  <xacro:include filename="$(find barista_robot_description)/xacro/standoff_rod.xacro"/>
-  <xacro:include filename="$(find barista_robot_description)/xacro/cup_holder_tray.xacro"/>
-  <xacro:include filename="$(find barista_robot_description)/xacro/laser_scanner.xacro"/>
-  <!-- Base -->
-  <link name="base_footprint"/>
-  <joint name="base_joint" type="fixed">
-    <parent link="base_footprint"/>
-    <child link="base_link"/>
-    <origin xyz="0 0 0.1127"/>
+<xacro:include filename="$(find barista_robot_description)/xacro/box_bot.gazebo.xacro" />
+<xacro:include filename="$(find barista_robot_description)/xacro/drive_wheel.xacro" />
+<xacro:include filename="$(find barista_robot_description)/xacro/caster_wheel.xacro" />
+<xacro:property name="body_width" value="0.1"/>
+<xacro:property name="body_lenght" value="0.1"/>
+<xacro:property name="body_height" value="0.1"/>
+<link name="base_link">
+  </link>
+  <joint name="base_link_joint" type="fixed">
+    <origin rpy="0 0 0" xyz="0 0 0" />
+    <parent link="base_link" />
+    <child link="chassis" />
   </joint>
-  <link name="base_link">
-    <visual><geometry><cylinder radius="0.178" length="0.155"/></geometry></visual>
-    <collision><geometry><cylinder radius="0.178" length="0.155"/></geometry></collision>
-    <inertial><mass value="10.0"/></inertial>
+  <link name="chassis">
+    <visual>
+      <geometry>
+        <box size="${body_width} ${body_lenght} ${body_height}"/>
+      </geometry>
+    </visual>
+    <collision>
+      <geometry>
+        <box size="${body_width} ${body_lenght} ${body_height}"/>
+      </geometry>
+    </collision>
+    <inertial>
+      <mass value="0.5"/>
+      <origin rpy="0 0 0" xyz="0 0 0"/>
+      <inertia ixx="0.0008333333333333335" ixy="0" ixz="0" iyy="0.0008333333333333335" iyz="0" izz="0.0008333333333333335"/>
+    </inertial>
   </link>
-  <!-- Wheels -->
-  <xacro:drive_wheel side="left" parent="base_link" xyz="0 0.15 -0.0775" rpy="-1.57 0 0" axis="0 0 1"/>
-  <xacro:drive_wheel side="right" parent="base_link" xyz="0 -0.15 -0.0775" rpy="1.57 0 0" axis="0 0 -1"/>
-  <!-- Casters -->
-  <xacro:caster_wheel name="front_caster" parent="base_link" xyz="0.1 0.0 -0.0775"/>
-  <xacro:caster_wheel name="back_caster" parent="base_link" xyz="-0.1 0.0 -0.0775"/>
-  <!-- Standoffs -->
-  <xacro:standoff_rod name="Standoff_Rod_1" parent="base_link" xyz="0.1 0.1 0.1875"/>
-  <xacro:standoff_rod name="Standoff_Rod_2" parent="base_link" xyz="-0.1 -0.1 0.1875"/>
-  <xacro:standoff_rod name="Standoff_Rod_3" parent="base_link" xyz="0.1 -0.1 0.1875"/>
-  <xacro:standoff_rod name="Standoff_Rod_4" parent="base_link" xyz="-0.1 0.1 0.1875"/>
-  <!-- Tray -->
-  <xacro:cup_holder_tray parent="base_link" xyz="0 0 0.3425"/>
-  <!-- Optional laser -->
-  <!-- <xacro:if value="${include_laser}">
-    <xacro:laser_scanner parent="base_link" xyz="0.14 0.0 0.0775"/>
-  </xacro:if> -->
-  <xacro:laser_scanner parent="base_link" xyz="0.14 0.0 0.0775"/>
 </robot>

File: xacro/caster_wheel.xacro (robot description, xacro)
@@ -1,5 +1,170 @@
 <?xml version="1.0"?>
 <robot xmlns:xacro="http://www.ros.org/wiki/xacro" name="barista_bot">
-  <xacro:macro name="caster_wheel" params="name parent xyz">
+ <!-- Caster Wheel Front -->
+  <link name="front_yaw_link">
+      <visual>
+        <origin rpy="0 1.5707 1.5707" xyz="0 0 0"/>
+        <geometry>
+          <cylinder length="0.001" radius="0.0045000000000000005"/>
+        </geometry>
+      </visual>
+      <collision>
+        <origin rpy="0 1.5707 1.5707" xyz="0 0 0"/>
+        <geometry>
+          <cylinder length="0.001" radius="0.0045000000000000005"/>
+        </geometry>
+      </collision>
+      <inertial>
+          <origin rpy="0 1.5707 1.5707" xyz="0 0 0"/>
+          <mass value="0.001"/>
+          <inertia ixx="5.145833333333334e-09" ixy="0" ixz="0" iyy="5.145833333333334e-09" iyz="0" izz="1.0125000000000003e-08"/>
+      </inertial>
+  </link>
+  <joint name="front_yaw_joint" type="continuous">
+    <origin rpy="0 0 0" xyz="0.04 0 -0.05" />
+    <parent link="chassis" />
+    <child link="front_yaw_link" />
+    <axis xyz="0 0 1" />
+    <limit effort="1000.0" velocity="100.0" />
+    <dynamics damping="0.0" friction="0.1"/>
+  </joint>
+  <link name="front_roll_link">
+      <visual>
+        <origin rpy="0 1.5707 1.5707" xyz="0 0 0"/>
+        <geometry>
+          <cylinder length="0.001" radius="0.0045000000000000005"/>
+        </geometry>
+      </visual>
+      <collision>
+        <origin rpy="0 1.5707 1.5707" xyz="0 0 0"/>
+        <geometry>
+          <cylinder length="0.001" radius="0.0045000000000000005"/>
+        </geometry>
+      </collision>
+      <inertial>
+          <origin rpy="0 1.5707 1.5707" xyz="0 0 0"/>
+          <mass value="0.001"/>
+          <inertia ixx="5.145833333333334e-09" ixy="0" ixz="0" iyy="5.145833333333334e-09" iyz="0" izz="1.0125000000000003e-08"/>
+      </inertial>
+  </link>
+  <joint name="front_roll_joint" type="continuous">
+    <origin rpy="0 0 0" xyz="0 0 0" />
+    <parent link="front_yaw_link" />
+    <child link="front_roll_link" />
+    <axis xyz="1 0 0" />
+    <limit effort="1000.0" velocity="100.0" />
+    <dynamics damping="0.0" friction="0.1"/>
+  </joint>
+  <link name="front_pitch_link">
+    <visual>
+      <origin rpy="0 1.5707 1.5707" xyz="0 0 0"/>
+      <geometry>
+        <sphere radius="0.010"/>
+      </geometry>
+    </visual>
+    <collision>
+      <origin rpy="0 1.5707 1.5707" xyz="0 0 0"/>
+      <geometry>
+        <sphere radius="0.010"/>
+      </geometry>
+    </collision>
+    <inertial>
+        <origin rpy="0 1.5707 1.5707" xyz="0 0 0"/>
+        <mass value="0.001"/>
+        <inertia ixx="4e-08" ixy="0" ixz="0" iyy="4e-08" iyz="0" izz="4e-08"/>
+    </inertial>
+  </link>
+  <joint name="front_pitch_joint" type="continuous">
+    <origin rpy="0 0 0" xyz="0 0 0" />
+    <parent link="front_roll_link" />
+    <child link="front_pitch_link" />
+    <axis xyz="0 1 0" />
+    <limit effort="1000.0" velocity="100.0" />
+    <dynamics damping="0.0" friction="0.1"/>
+  </joint>
+<!-- Caster Wheel Back -->
+  <link name="back_yaw_link">
+    <visual>
+        <origin rpy="0 1.5707 1.5707" xyz="0 0 0"/>
+        <geometry>
+          <cylinder length="0.001" radius="0.0045000000000000005"/>
+        </geometry>
+      </visual>
+      <collision>
+        <origin rpy="0 1.5707 1.5707" xyz="0 0 0"/>
+        <geometry>
+          <cylinder length="0.001" radius="0.0045000000000000005"/>
+        </geometry>
+      </collision>
+      <inertial>
+          <origin rpy="0 1.5707 1.5707" xyz="0 0 0"/>
+          <mass value="0.001"/>
+          <inertia ixx="5.145833333333334e-09" ixy="0" ixz="0" iyy="5.145833333333334e-09" iyz="0" izz="1.0125000000000003e-08"/>
+      </inertial>
+  </link>
+  <joint name="back_yaw_joint" type="continuous">
+    <origin rpy="0 0 0" xyz="-0.04 0 -0.05" />
+    <parent link="chassis" />
+    <child link="back_yaw_link" />
+    <axis xyz="0 0 1" />
+    <limit effort="1000.0" velocity="100.0" />
+    <dynamics damping="0.0" friction="0.1"/>
+  </joint>
+  <link name="back_roll_link">
+      <visual>
+        <origin rpy="0 1.5707 1.5707" xyz="0 0 0"/>
+        <geometry>
+          <cylinder length="0.001" radius="0.0045000000000000005"/>
+        </geometry>
+      </visual>
+      <collision>
+        <origin rpy="0 1.5707 1.5707" xyz="0 0 0"/>
+        <geometry>
+          <cylinder length="0.001" radius="0.0045000000000000005"/>
+        </geometry>
+      </collision>
+      <inertial>
+          <origin rpy="0 1.5707 1.5707" xyz="0 0 0"/>
+          <mass value="0.001"/>
+          <inertia ixx="5.145833333333334e-09" ixy="0" ixz="0" iyy="5.145833333333334e-09" iyz="0" izz="1.0125000000000003e-08"/>
+      </inertial>
+  </link>
+  <joint name="back_roll_joint" type="continuous">
+    <origin rpy="0 0 0" xyz="0 0 0" />
+    <parent link="back_yaw_link" />
+    <child link="back_roll_link" />
+    <axis xyz="1 0 0" />
+    <limit effort="1000.0" velocity="100.0" />
+    <dynamics damping="0.0" friction="0.1"/>
+  </joint>
+  <link name="back_pitch_link">
+    <visual>
+      <origin rpy="0 1.5707 1.5707" xyz="0 0 0"/>
+      <geometry>
+        <sphere radius="0.010"/>
+      </geometry>
+    </visual>
+    <collision>
+      <origin rpy="0 1.5707 1.5707" xyz="0 0 0"/>
+      <geometry>
+        <sphere radius="0.010"/>
+      </geometry>
+    </collision>
+    <inertial>
+        <origin rpy="0 1.5707 1.5707" xyz="0 0 0"/>
+        <mass value="0.001"/>
+        <inertia ixx="4e-08" ixy="0" ixz="0" iyy="4e-08" iyz="0" izz="4e-08"/>
+    </inertial>
+  </link>
+  <joint name="back_pitch_joint" type="continuous">
+    <origin rpy="0 0 0" xyz="0 0 0" />
+    <parent link="back_roll_link" />
+    <child link="back_pitch_link" />
+    <axis xyz="0 1 0" />
+    <limit effort="1000.0" velocity="100.0" />
+    <dynamics damping="0.0" friction="0.1"/>
+  </joint>
+</robot>
+  <!-- <xacro:macro name="caster_wheel" params="name parent xyz">
     <joint name="${name}_joint" type="fixed">
       <parent link="${parent}"/>
@@ -13,3 +178,3 @@
     </link>
   </xacro:macro>
-</robot>
+</robot> -->

File: xacro/drive_wheel.xacro (robot description, xacro)
@@ -1,5 +1,50 @@
 <?xml version="1.0"?>
 <robot xmlns:xacro="http://www.ros.org/wiki/xacro" name="barista_bot">
-  <xacro:macro name="drive_wheel" params="side parent xyz rpy axis">
+<xacro:property name="wheel_width" value="0.001"/>
+<xacro:property name="wheel_radius" value="0.035"/>
+<!-- Wheel Macro -->
+<xacro:macro name="wheel" params="wheel_name">
+  <link name="${wheel_name}">
+      <visual>
+        <origin rpy="0 1.5707 1.5707" xyz="0 0 0"/>
+        <geometry>
+          <cylinder length="${wheel_width}" radius="${wheel_radius}"/>
+        </geometry>
+      </visual>
+      <collision>
+        <origin rpy="0 1.5707 1.5707" xyz="0 0 0"/>
+        <geometry>
+          <cylinder length="${wheel_width}" radius="${wheel_radius}"/>
+        </geometry>
+      </collision>
+      <inertial>
+        <origin rpy="0 1.5707 1.5707" xyz="0 0 0"/>
+        <mass value="0.05"/>
+        <inertia ixx="1.531666666666667e-05" ixy="0" ixz="0" iyy="1.531666666666667e-05" iyz="0" izz="3.0625000000000006e-05"/>
+      </inertial>
+  </link>
+</xacro:macro>
+  <!-- Wheel Left -->
+ <xacro:wheel wheel_name="left_wheel" />
+  <!-- Wheel Right -->
+  <xacro:wheel wheel_name="right_wheel" />
+  <joint name="joint_left_wheel" type="continuous">
+    <origin rpy="0 0 0" xyz="0 0.05 -0.025"/>
+    <child link="left_wheel"/>
+    <parent link="chassis"/>
+    <axis rpy="0 0 0" xyz="0 1 0"/>
+    <limit effort="10000" velocity="1000"/>
+    <joint_properties damping="1.0" friction="1.0"/>
+  </joint>
+  <joint name="joint_right_wheel" type="continuous">
+    <origin rpy="0 0 0" xyz="0 -0.05 -0.025"/>
+    <child link="right_wheel"/>
+    <parent link="chassis"/>
+    <axis rpy="0 0 0" xyz="0 1 0"/>
+    <limit effort="10000" velocity="1000"/>
+    <joint_properties damping="1.0" friction="1.0"/>
+  </joint>
+</robot>
+  <!-- <xacro:macro name="drive_wheel" params="side parent xyz rpy axis">
     <joint name="${side}_wheel_joint" type="continuous">
       <parent link="${parent}"/>
@@ -14,3 +59,3 @@
     </link>
   </xacro:macro>
-</robot>
+</robot> -->
