Commit message: commit for task2 again

File: xacro/barista_robot_model.urdf.xacro (robot description, xacro)
@@ -1,33 +1,53 @@
 <?xml version="1.0"?>
 <robot xmlns:xacro="http://www.ros.org/wiki/xacro" name="barista_bot">
-<xacro:include filename="$(find barista_robot_description)/xacro/box_bot.gazebo.xacro" />
+<xacro:include filename="$(find barista_robot_description)/xacro/barista_bot.gazebo.xacro" />
 <xacro:include filename="$(find barista_robot_description)/xacro/drive_wheel.xacro" />
 <xacro:include filename="$(find barista_robot_description)/xacro/caster_wheel.xacro" />
-<xacro:property name="body_width" value="0.1"/>
-<xacro:property name="body_lenght" value="0.1"/>
-<xacro:property name="body_height" value="0.1"/>
-<link name="base_link">
-  </link>
-  <joint name="base_link_joint" type="fixed">
-    <origin rpy="0 0 0" xyz="0 0 0" />
-    <parent link="base_link" />
-    <child link="chassis" />
-  </joint>
-  <link name="chassis">
-    <visual>
-      <geometry>
-        <box size="${body_width} ${body_lenght} ${body_height}"/>
-      </geometry>
-    </visual>
-    <collision>
-      <geometry>
-        <box size="${body_width} ${body_lenght} ${body_height}"/>
-      </geometry>
-    </collision>
-    <inertial>
-      <mass value="0.5"/>
-      <origin rpy="0 0 0" xyz="0 0 0"/>
-      <inertia ixx="0.0008333333333333335" ixy="0" ixz="0" iyy="0.0008333333333333335" iyz="0" izz="0.0008333333333333335"/>
-    </inertial>
-  </link>
+<xacro:include filename="$(find barista_robot_description)/xacro/cup_holder_tray.xacro" />
+<xacro:include filename="$(find barista_robot_description)/xacro/standoff_rod.xacro" />
+<xacro:include filename="$(find barista_robot_description)/xacro/laser_scanner.xacro" />
+    <material name="white">
+        <color rgba="1 1 1 1" />
+    </material>
+    <material name="orange">
+        <color rgba="1 0.3 0.1 1"/>
+    </material>
+    <material name="blue">
+        <color rgba="0.2 0.2 1 1"/>
+    </material>
+    <material name="black">
+        <color rgba="0 0 0 1"/>
+    </material>
+    <material name="red">
+        <color rgba="1 0 0 1"/>
+    </material>
+    <!-- BASE FOOTPRINT-->
+    <link name="base_footprint">
+    </link>
+    <!-- BASE LINK -->
+    <joint name="base_joint" type="fixed">
+        <parent link="base_footprint"/>
+        <child link="base_link"/>
+        <origin xyz="0 0 0.1127"/>
+    </joint>
+    <link name="base_link">
+        <inertial>
+            <mass value="10.0" />
+            <origin xyz="0 0 0" rpy="0 0 0" />
+            <inertia ixx="0.09923083333333334" ixy="0.0" ixz="0.0" iyy="0.09923083333333334" iyz="0.0" izz="0.15841999999999998" />
+        </inertial>
+        <visual>
+            <origin xyz="0 0 0"/>
+            <geometry>
+                <cylinder radius="0.178" length="0.155"/>
+            </geometry>
+            <material name="blue"/>
+        </visual>
+        <collision>
+            <origin xyz="0 0 0"/>
+            <geometry>
+                <cylinder radius="0.178" length="0.155"/>
+            </geometry>
+        </collision>
+    </link>
 </robot>

File: xacro/caster_wheel.xacro (robot description, xacro)
@@ -1,180 +1,51 @@
 <?xml version="1.0"?>
 <robot xmlns:xacro="http://www.ros.org/wiki/xacro" name="barista_bot">
- <!-- Caster Wheel Front -->
-  <link name="front_yaw_link">
-      <visual>
-        <origin rpy="0 1.5707 1.5707" xyz="0 0 0"/>
-        <geometry>
-          <cylinder length="0.001" radius="0.0045000000000000005"/>
-        </geometry>
-      </visual>
-      <collision>
-        <origin rpy="0 1.5707 1.5707" xyz="0 0 0"/>
-        <geometry>
-          <cylinder length="0.001" radius="0.0045000000000000005"/>
-        </geometry>
-      </collision>
-      <inertial>
-          <origin rpy="0 1.5707 1.5707" xyz="0 0 0"/>
-          <mass value="0.001"/>
-          <inertia ixx="5.145833333333334e-09" ixy="0" ixz="0" iyy="5.145833333333334e-09" iyz="0" izz="1.0125000000000003e-08"/>
-      </inertial>
-  </link>
-  <joint name="front_yaw_joint" type="continuous">
-    <origin rpy="0 0 0" xyz="0.04 0 -0.05" />
-    <parent link="chassis" />
-    <child link="front_yaw_link" />
-    <axis xyz="0 0 1" />
-    <limit effort="1000.0" velocity="100.0" />
-    <dynamics damping="0.0" friction="0.1"/>
-  </joint>
-  <link name="front_roll_link">
-      <visual>
-        <origin rpy="0 1.5707 1.5707" xyz="0 0 0"/>
-        <geometry>
-          <cylinder length="0.001" radius="0.0045000000000000005"/>
-        </geometry>
-      </visual>
-      <collision>
-        <origin rpy="0 1.5707 1.5707" xyz="0 0 0"/>
-        <geometry>
-          <cylinder length="0.001" radius="0.0045000000000000005"/>
-        </geometry>
-      </collision>
-      <inertial>
-          <origin rpy="0 1.5707 1.5707" xyz="0 0 0"/>
-          <mass value="0.001"/>
-          <inertia ixx="5.145833333333334e-09" ixy="0" ixz="0" iyy="5.145833333333334e-09" iyz="0" izz="1.0125000000000003e-08"/>
-      </inertial>
-  </link>
-  <joint name="front_roll_joint" type="continuous">
-    <origin rpy="0 0 0" xyz="0 0 0" />
-    <parent link="front_yaw_link" />
-    <child link="front_roll_link" />
-    <axis xyz="1 0 0" />
-    <limit effort="1000.0" velocity="100.0" />
-    <dynamics damping="0.0" friction="0.1"/>
-  </joint>
-  <link name="front_pitch_link">
-    <visual>
-      <origin rpy="0 1.5707 1.5707" xyz="0 0 0"/>
-      <geometry>
-        <sphere radius="0.010"/>
-      </geometry>
-    </visual>
-    <collision>
-      <origin rpy="0 1.5707 1.5707" xyz="0 0 0"/>
-      <geometry>
-        <sphere radius="0.010"/>
-      </geometry>
-    </collision>
-    <inertial>
-        <origin rpy="0 1.5707 1.5707" xyz="0 0 0"/>
-        <mass value="0.001"/>
-        <inertia ixx="4e-08" ixy="0" ixz="0" iyy="4e-08" iyz="0" izz="4e-08"/>
-    </inertial>
-  </link>
-  <joint name="front_pitch_joint" type="continuous">
-    <origin rpy="0 0 0" xyz="0 0 0" />
-    <parent link="front_roll_link" />
-    <child link="front_pitch_link" />
-    <axis xyz="0 1 0" />
-    <limit effort="1000.0" velocity="100.0" />
-    <dynamics damping="0.0" friction="0.1"/>
-  </joint>
-<!-- Caster Wheel Back -->
-  <link name="back_yaw_link">
-    <visual>
-        <origin rpy="0 1.5707 1.5707" xyz="0 0 0"/>
-        <geometry>
-          <cylinder length="0.001" radius="0.0045000000000000005"/>
-        </geometry>
-      </visual>
-      <collision>
-        <origin rpy="0 1.5707 1.5707" xyz="0 0 0"/>
-        <geometry>
-          <cylinder length="0.001" radius="0.0045000000000000005"/>
-        </geometry>
-      </collision>
-      <inertial>
-          <origin rpy="0 1.5707 1.5707" xyz="0 0 0"/>
-          <mass value="0.001"/>
-          <inertia ixx="5.145833333333334e-09" ixy="0" ixz="0" iyy="5.145833333333334e-09" iyz="0" izz="1.0125000000000003e-08"/>
-      </inertial>
-  </link>
-  <joint name="back_yaw_joint" type="continuous">
-    <origin rpy="0 0 0" xyz="-0.04 0 -0.05" />
-    <parent link="chassis" />
-    <child link="back_yaw_link" />
-    <axis xyz="0 0 1" />
-    <limit effort="1000.0" velocity="100.0" />
-    <dynamics damping="0.0" friction="0.1"/>
-  </joint>
-  <link name="back_roll_link">
-      <visual>
-        <origin rpy="0 1.5707 1.5707" xyz="0 0 0"/>
-        <geometry>
-          <cylinder length="0.001" radius="0.0045000000000000005"/>
-        </geometry>
-      </visual>
-      <collision>
-        <origin rpy="0 1.5707 1.5707" xyz="0 0 0"/>
-        <geometry>
-          <cylinder length="0.001" radius="0.0045000000000000005"/>
-        </geometry>
-      </collision>
-      <inertial>
-          <origin rpy="0 1.5707 1.5707" xyz="0 0 0"/>
-          <mass value="0.001"/>
-          <inertia ixx="5.145833333333334e-09" ixy="0" ixz="0" iyy="5.145833333333334e-09" iyz="0" izz="1.0125000000000003e-08"/>
-      </inertial>
-  </link>
-  <joint name="back_roll_joint" type="continuous">
-    <origin rpy="0 0 0" xyz="0 0 0" />
-    <parent link="back_yaw_link" />
-    <child link="back_roll_link" />
-    <axis xyz="1 0 0" />
-    <limit effort="1000.0" velocity="100.0" />
-    <dynamics damping="0.0" friction="0.1"/>
-  </joint>
-  <link name="back_pitch_link">
-    <visual>
-      <origin rpy="0 1.5707 1.5707" xyz="0 0 0"/>
-      <geometry>
-        <sphere radius="0.010"/>
-      </geometry>
-    </visual>
-    <collision>
-      <origin rpy="0 1.5707 1.5707" xyz="0 0 0"/>
-      <geometry>
-        <sphere radius="0.010"/>
-      </geometry>
-    </collision>
-    <inertial>
-        <origin rpy="0 1.5707 1.5707" xyz="0 0 0"/>
-        <mass value="0.001"/>
-        <inertia ixx="4e-08" ixy="0" ixz="0" iyy="4e-08" iyz="0" izz="4e-08"/>
-    </inertial>
-  </link>
-  <joint name="back_pitch_joint" type="continuous">
-    <origin rpy="0 0 0" xyz="0 0 0" />
-    <parent link="back_roll_link" />
-    <child link="back_pitch_link" />
-    <axis xyz="0 1 0" />
-    <limit effort="1000.0" velocity="100.0" />
-    <dynamics damping="0.0" friction="0.1"/>
-  </joint>
+<!-- FRONT CASTER WHEEL -->
+    <joint name="front_caster_wheel_joint" type="fixed">
+        <parent link="base_link"/>
+        <child link="front_caster"/>
+        <origin xyz="0.1 0.0 -0.0775" rpy="0 0 0" />
+        <axis xyz="0 0 0"/>
+    </joint>
+    <link name="front_caster">
+        <visual>
+            <geometry>
+                <sphere radius="0.0352"/>
+            </geometry>
+        </visual>
+        <collision>
+            <geometry>
+                <sphere radius="0.0352"/>
+            </geometry>
+        </collision>
+        <inertial>
+            <mass value="0.5" />
+            <origin xyz="0 0 0" rpy="0 0 0" />
+            <inertia ixx="9.479166666666669e-06" ixy="0.0" ixz="0.0" iyy="9.479166666666669e-06" iyz="0.0" izz="1.5625000000000004e-05" />
+        </inertial>
+    </link>
+    <!-- REAR CASTER WHEEL -->
+    <joint name="rear_caster_wheel_joint" type="fixed">
+        <parent link="base_link"/>
+        <child link="back_caster"/>
+        <origin xyz="-0.1 0.0 -0.0775" rpy="0 0 0" />
+        <axis xyz="0 0 0"/>
+    </joint>
+    <link name="back_caster">
+        <visual>
+            <geometry>
+                <sphere radius="0.0352"/>
+            </geometry>
+        </visual>
+        <collision>
+            <geometry>
+                <sphere radius="0.0352"/>
+            </geometry>
+        </collision>
+        <inertial>
+            <mass value="0.5" />
+            <origin xyz="0 0 0" rpy="0 0 0" />
+            <inertia ixx="0.000247808" ixy="0.0" ixz="0.0" iyy="0.000247808" iyz="0.0" izz="0.000247808" />
+        </inertial>
+    </link>
 </robot>
-  <!-- <xacro:macro name="caster_wheel" params="name parent xyz">
-    <joint name="${name}_joint" type="fixed">
-      <parent link="${parent}"/>
-      <child link="${name}"/>
-      <origin xyz="${xyz}"/>
-    </joint>
-    <link name="${name}">
-      <visual><geometry><sphere radius="0.0352"/></geometry></visual>
-      <collision><geometry><sphere radius="0.0352"/></geometry></collision>
-      <inertial><mass value="0.5"/></inertial>
-    </link>
-  </xacro:macro>
-</robot> -->

File: xacro/cup_holder_tray.xacro (robot description, xacro)
@@ -1,15 +1,29 @@
 <?xml version="1.0"?>
 <robot xmlns:xacro="http://www.ros.org/wiki/xacro" name="barista_bot">
-  <xacro:macro name="cup_holder_tray" params="parent xyz">
+    <!-- Cup_Holder_Tray_link -->
     <joint name="Cup_Holder_Tray_Joint" type="fixed">
-      <parent link="${parent}"/>
-      <child link="Cup_Holder_Tray_link"/>
-      <origin xyz="${xyz}"/>
+        <parent link="base_link"/>
+        <child link="Cup_Holder_Tray_link"/>
+        <origin xyz="0 0 0.3425"/>
     </joint>
     <link name="Cup_Holder_Tray_link">
-      <visual><geometry><cylinder radius="0.160" length="0.090"/></geometry></visual>
-      <collision><geometry><cylinder radius="0.160" length="0.090"/></geometry></collision>
-      <inertial><mass value="8.0"/></inertial>
+        <inertial>
+            <mass value="8.0" />
+            <origin xyz="0 0 0" rpy="0 0 0" />
+                <inertia ixx="0.0566" ixy="0.0" ixz="0.0" iyy="0.0566" iyz="0.0" izz="0.1024" />
+        </inertial>
+        <visual>
+            <origin xyz="0 0 0"/>
+            <geometry>
+                <cylinder radius="0.160" length="0.090"/>
+            </geometry>
+            <material name="blue"/>
+        </visual>
+        <collision>
+            <origin xyz="0 0 0"/>
+            <geometry>
+                <cylinder radius="0.160" length="0.090"/>
+            </geometry>
+        </collision>
     </link>
-  </xacro:macro>
 </robot>

File: xacro/drive_wheel.xacro (robot description, xacro)
@@ -1,61 +1,57 @@
 <?xml version="1.0"?>
 <robot xmlns:xacro="http://www.ros.org/wiki/xacro" name="barista_bot">
-<xacro:property name="wheel_width" value="0.001"/>
-<xacro:property name="wheel_radius" value="0.035"/>
-<!-- Wheel Macro -->
-<xacro:macro name="wheel" params="wheel_name">
-  <link name="${wheel_name}">
-      <visual>
-        <origin rpy="0 1.5707 1.5707" xyz="0 0 0"/>
-        <geometry>
-          <cylinder length="${wheel_width}" radius="${wheel_radius}"/>
-        </geometry>
-      </visual>
-      <collision>
-        <origin rpy="0 1.5707 1.5707" xyz="0 0 0"/>
-        <geometry>
-          <cylinder length="${wheel_width}" radius="${wheel_radius}"/>
-        </geometry>
-      </collision>
-      <inertial>
-        <origin rpy="0 1.5707 1.5707" xyz="0 0 0"/>
-        <mass value="0.05"/>
-        <inertia ixx="1.531666666666667e-05" ixy="0" ixz="0" iyy="1.531666666666667e-05" iyz="0" izz="3.0625000000000006e-05"/>
-      </inertial>
-  </link>
-</xacro:macro>
-  <!-- Wheel Left -->
- <xacro:wheel wheel_name="left_wheel" />
-  <!-- Wheel Right -->
-  <xacro:wheel wheel_name="right_wheel" />
-  <joint name="joint_left_wheel" type="continuous">
-    <origin rpy="0 0 0" xyz="0 0.05 -0.025"/>
-    <child link="left_wheel"/>
-    <parent link="chassis"/>
-    <axis rpy="0 0 0" xyz="0 1 0"/>
-    <limit effort="10000" velocity="1000"/>
-    <joint_properties damping="1.0" friction="1.0"/>
-  </joint>
-  <joint name="joint_right_wheel" type="continuous">
-    <origin rpy="0 0 0" xyz="0 -0.05 -0.025"/>
-    <child link="right_wheel"/>
-    <parent link="chassis"/>
-    <axis rpy="0 0 0" xyz="0 1 0"/>
-    <limit effort="10000" velocity="1000"/>
-    <joint_properties damping="1.0" friction="1.0"/>
-  </joint>
+    <!-- LEFT WHEEL LINK -->
+    <joint name="left_wheel_joint" type="continuous">
+        <parent link="base_link"/>
+        <child link="left_wheel"/>
+        <origin xyz="0 0.15 -0.0775" rpy="-1.57 0 0" />
+        <axis xyz="0 0 1"/>
+    </joint>
+    <link name="left_wheel">
+        <inertial>
+            <mass value="1.5" />
+            <origin xyz="0 0 0" rpy="-1.57 0 0" />
+            <inertia ixx=" 0.000517685" ixy="0.0" ixz="0.0" iyy= "0.000517685" iyz="0.0" izz="0.00092928" />
+        </inertial>
+        <visual>
+            <origin xyz="0 0 0" rpy="0 0 0"/>
+            <geometry>
+                <cylinder radius="0.0352" length="0.0206"/>
+            </geometry>
+            <material name="black"/>
+        </visual>
+        <collision>
+            <origin xyz="0 0 0" rpy="0 0 0"/>
+            <geometry>
+                <cylinder radius="0.0352" length="0.0206"/>
+            </geometry>
+        </collision>
+    </link>
+    <!-- RIGHT WHEEL LINK -->
+    <joint name="right_wheel_joint" type="continuous">
+        <parent link="base_link"/>
+        <child link="right_wheel"/>
+        <origin xyz="0 -0.15 -0.0775" rpy="1.57 0 0" />
+        <axis xyz="0 0 -1"/>
+    </joint>
+    <link name="right_wheel">
+        <inertial>
+            <mass value="1.5" />
+            <origin xyz="0 0 0" rpy="-1.575 0 0" />
+        <inertia ixx=" 0.000517685" ixy="0.0" ixz="0.0" iyy= "0.000517685" iyz="0.0" izz="0.00092928" />
+        </inertial>
+        <visual>
+            <origin xyz="0 0 0" rpy="0 0 0"/>
+            <geometry>
+                <cylinder radius="0.0352" length="0.0206"/>
+            </geometry>
+            <material name="black"/>
+        </visual>
+        <collision>
+            <origin xyz="0 0 0" rpy="0 0 0"/>
+            <geometry>
+                <cylinder radius="0.0352" length="0.0206"/>
+            </geometry>
+        </collision>
+    </link>
 </robot>
-  <!-- <xacro:macro name="drive_wheel" params="side parent xyz rpy axis">
-    <joint name="${side}_wheel_joint" type="continuous">
-      <parent link="${parent}"/>
-      <child link="${side}_wheel"/>
-      <origin xyz="${xyz}" rpy="${rpy}"/>
-      <axis xyz="${axis}"/>
-    </joint>
-    <link name="${side}_wheel">
-      <visual><geometry><cylinder radius="0.0352" length="0.0206"/></geometry></visual>
-      <collision><geometry><cylinder radius="0.0352" length="0.0206"/></geometry></collision>
-      <inertial><mass value="1.5"/></inertial>
-    </link>
-  </xacro:macro>
-</robot> -->

File: xacro/laser_scanner.xacro (robot description, xacro)
@@ -1,15 +1,31 @@
 <?xml version="1.0"?>
 <robot xmlns:xacro="http://www.ros.org/wiki/xacro" name="barista_bot">
-  <xacro:macro name="laser_scanner" params="parent xyz">
+    <!-- Laser scan -->
     <joint name="front_laser_joint" type="fixed">
-      <parent link="${parent}"/>
-      <child link="front_laser"/>
-      <origin xyz="${xyz}"/>
+        <parent link="base_link"/>
+        <child link="front_laser"/>
+        <origin xyz="0.14 0 0.078" rpy="0 0 0" />
+        <axis xyz="0 0 0"/>
     </joint>
     <link name="front_laser">
-      <visual><geometry><cylinder radius="0.025" length="0.06"/></geometry></visual>
-      <collision><geometry><cylinder radius="0.025" length="0.06"/></geometry></collision>
-      <inertial><mass value="0.05"/></inertial>
+        <inertial>
+            <origin xyz="0 0 0" rpy="0 0 0" />
+            <mass value="0.05" />
+            <inertia ixx="0.000252666666667" ixy="0" ixz="0" iyy="0.000252666666667" iyz="0" izz="0.0005"/>
+        </inertial>
+        <visual>
+            <origin xyz="0 0 0" rpy="0 0 0" />
+            <geometry>
+                <mesh filename="package://barista_robot_description/meshes/sick_s3000.dae" scale="0.2 0.2 0.2"/>
+                <!-- <cylinder radius="0.025" length="0.02"/> -->
+            </geometry>
+            <material name="red"/>
+        </visual>
+        <collision>
+            <origin xyz="0 0 0" rpy="0 0 0"/>
+            <geometry>
+                <cylinder radius="0.025" length="0.02"/>
+            </geometry>
+        </collision>
     </link>
-  </xacro:macro>
 </robot>

File: xacro/standoff_rod.xacro (robot description, xacro)
@@ -1,15 +1,107 @@
 <?xml version="1.0"?>
 <robot xmlns:xacro="http://www.ros.org/wiki/xacro" name="barista_bot">
-  <xacro:macro name="standoff_rod" params="name parent xyz">
-    <joint name="${name}_Joint" type="fixed">
-      <parent link="${parent}"/>
-      <child link="${name}_link"/>
-      <origin xyz="${xyz}"/>
+    <!-- Standoff_Rod_1_link -->
+    <joint name="Standoff_Rod_1_Joint" type="fixed">
+        <parent link="base_link"/>
+        <child link="Standoff_Rod_1_link"/>
+        <origin xyz="0.1 0.1 0.1875"/>
     </joint>
-    <link name="${name}_link">
-      <visual><geometry><cylinder radius="0.01" length="0.22"/></geometry></visual>
-      <collision><geometry><cylinder radius="0.01" length="0.22"/></geometry></collision>
-      <inertial><mass value="0.5"/></inertial>
+    <link name="Standoff_Rod_1_link">
+        <inertial>
+            <mass value="0.5" />
+            <origin xyz="0 0 0" rpy="0 0 0" />
+            <inertia ixx="0.0020291666666666665" ixy="0.0" ixz="0.0" iyy="0.0020291666666666665" iyz="0.0" izz="2.5e-05" />
+        </inertial>
+        <visual>
+            <origin xyz="0 0 0"/>
+            <geometry>
+                <cylinder radius="0.01" length="0.22"/>
+            </geometry>
+            <material name="white"/>
+        </visual>
+        <collision>
+            <origin xyz="0 0 0"/>
+            <geometry>
+                <cylinder radius="0.01" length="0.22"/>
+            </geometry>
+        </collision>
     </link>
-  </xacro:macro>
+    <!-- Standoff_Rod_2_link -->
+    <joint name="Standoff_Rod_2_Joint" type="fixed">
+        <parent link="base_link"/>
+        <child link="Standoff_Rod_2_link"/>
+        <origin xyz="-0.1 -0.1 0.1875"/>
+    </joint>
+    <link name="Standoff_Rod_2_link">
+        <inertial>
+            <mass value="0.5" />
+            <origin xyz="0 0 0" rpy="0 0 0" />
+            <inertia ixx="0.0020291666666666665" ixy="0.0" ixz="0.0" iyy="0.0020291666666666665" iyz="0.0" izz="2.5e-05" />
+        </inertial>
+        <visual>
+            <origin xyz="0 0 0"/>
+            <geometry>
+                <cylinder radius="0.01" length="0.22"/>
+            </geometry>
+            <material name="white"/>
+        </visual>
+        <collision>
+            <origin xyz="0 0 0"/>
+            <geometry>
+                <cylinder radius="0.01" length="0.22"/>
+            </geometry>
+        </collision>
+    </link>
+    <!-- Standoff_Rod_3_link -->
+    <joint name="Standoff_Rod_3_Joint" type="fixed">
+        <parent link="base_link"/>
+        <child link="Standoff_Rod_3_link"/>
+        <origin xyz="0.1 -0.1 0.1875"/>
+    </joint>
+    <link name="Standoff_Rod_3_link">
+        <inertial>
+            <mass value="0.5" />
+            <origin xyz="0 0 0" rpy="0 0 0" />
+            <inertia ixx="0.0020291666666666665" ixy="0.0" ixz="0.0" iyy="0.0020291666666666665" iyz="0.0" izz="2.5e-05" />
+        </inertial>
+        <visual>
+            <origin xyz="0 0 0"/>
+            <geometry>
+                <cylinder radius="0.01" length="0.22"/>
+            </geometry>
+            <material name="white"/>
+        </visual>
+        <collision>
+            <origin xyz="0 0 0"/>
+            <geometry>
+                <cylinder radius="0.01" length="0.22"/>
+            </geometry>
+        </collision>
+    </link>
+    <!-- Standoff_Rod_4_link -->
+    <joint name="Standoff_Rod_4_Joint" type="fixed">
+        <parent link="base_link"/>
+        <child link="Standoff_Rod_4_link"/>
+        <origin xyz="-0.1 0.1 0.1875"/>
+    </joint>
+    <link name="Standoff_Rod_4_link">
+        <inertial>
+            <mass value="0.5" />
+            <origin xyz="0 0 0" rpy="0 0 0" />
+            <inertia ixx="0.0020291666666666665" ixy="0.0" ixz="0.0" iyy="0.0020291666666666665" iyz="0.0" izz="2.5e-05" />
+        </inertial>
+        <visual>
+            <origin xyz="0 0 0"/>
+            <geometry>
+                <cylinder radius="0.01" length="0.22"/>
+            </geometry>
+            <material name="white"/>
+        </visual>
+        <collision>
+            <origin xyz="0 0 0"/>
+            <geometry>
+                <cylinder radius="0.01" length="0.22"/>
+            </geometry>
+        </collision>
+    </link>
 </robot>
