Commit message: rods positioned are corrected, xacro files are reorganzed, include laser is done yet

File: xacro/barista_robot_model.urdf.xacro (robot description, xacro)
@@ -1,29 +1,15 @@
 <?xml version="1.0"?>
 <robot xmlns:xacro="http://www.ros.org/wiki/xacro" name="barista_bot">
-<xacro:include filename="$(find barista_robot_description)/xacro/barista_bot.gazebo.xacro" />
-<xacro:include filename="$(find barista_robot_description)/xacro/drive_wheel.xacro" />
-<xacro:include filename="$(find barista_robot_description)/xacro/caster_wheel.xacro" />
-<xacro:include filename="$(find barista_robot_description)/xacro/cup_holder_tray.xacro" />
-<xacro:include filename="$(find barista_robot_description)/xacro/standoff_rod.xacro" />
-<xacro:include filename="$(find barista_robot_description)/xacro/laser_scanner.xacro" />
-    <material name="white">
-        <color rgba="1 1 1 1" />
-    </material>
-    <material name="orange">
-        <color rgba="1 0.3 0.1 1"/>
-    </material>
-    <material name="blue">
-        <color rgba="0.2 0.2 1 1"/>
-    </material>
-    <material name="black">
-        <color rgba="0 0 0 1"/>
-    </material>
-    <material name="red">
-        <color rgba="1 0 0 1"/>
-    </material>
-    <!-- BASE FOOTPRINT-->
-    <link name="base_footprint">
-    </link>
-    <!-- BASE LINK -->
+    <!-- Arguments -->
+    <xacro:arg name="robot_name" default="barista_bot"/>
+    <xacro:arg name="include_laser" default="true"/>
+    <!-- Materials -->
+    <material name="white"><color rgba="1 1 1 1"/></material>
+    <material name="orange"><color rgba="1 0.3 0.1 1"/></material>
+    <material name="blue"><color rgba="0.2 0.2 1 1"/></material>
+    <material name="black"><color rgba="0 0 0 1"/></material>
+    <material name="red"><color rgba="1 0 0 1"/></material>
+    <!-- Base -->
+    <link name="base_footprint"/>
     <joint name="base_joint" type="fixed">
         <parent link="base_footprint"/>
@@ -33,21 +19,78 @@
     <link name="base_link">
         <inertial>
-            <mass value="10.0" />
-            <origin xyz="0 0 0" rpy="0 0 0" />
-            <inertia ixx="0.09923083333333334" ixy="0.0" ixz="0.0" iyy="0.09923083333333334" iyz="0.0" izz="0.15841999999999998" />
+        <mass value="10.0"/>
+        <origin xyz="0 0 0" rpy="0 0 0"/>
+        <inertia ixx="0.09923083333333334" ixy="0" ixz="0" iyy="0.09923083333333334" iyz="0" izz="0.15842"/>
         </inertial>
         <visual>
-            <origin xyz="0 0 0"/>
-            <geometry>
-                <cylinder radius="0.178" length="0.155"/>
-            </geometry>
-            <material name="blue"/>
+        <origin xyz="0 0 0"/>
+        <geometry><cylinder radius="0.178" length="0.155"/></geometry>
+        <material name="blue"/>
         </visual>
         <collision>
-            <origin xyz="0 0 0"/>
-            <geometry>
-                <cylinder radius="0.178" length="0.155"/>
-            </geometry>
+        <origin xyz="0 0 0"/>
+        <geometry><cylinder radius="0.178" length="0.155"/></geometry>
         </collision>
     </link>
+    <gazebo reference="base_link"><material>Gazebo/Blue</material></gazebo>
+    <!-- Include modular components -->
+    <xacro:include filename="$(find barista_robot_description)/xacro/cup_holder_tray.xacro"/>
+    <xacro:include filename="$(find barista_robot_description)/xacro/standoff_rod.xacro"/>
+    <xacro:include filename="$(find barista_robot_description)/xacro/drive_wheel.xacro"/>
+    <xacro:include filename="$(find barista_robot_description)/xacro/caster_wheel.xacro"/>
+    <xacro:include filename="$(find barista_robot_description)/xacro/laser_scanner.xacro"/>
+    <!-- Add parts with parameters -->
+    <xacro:cup_holder_tray parent="base_link"/>
+    <!-- 4 standoff rods -->
+    <xacro:standoff_rod name="Standoff_Rod_1" parent="base_link" xyz="0.05 0.14 0.1875"/>
+    <xacro:standoff_rod name="Standoff_Rod_2" parent="base_link" xyz="-0.05 -0.14 0.1875"/>
+    <xacro:standoff_rod name="Standoff_Rod_3" parent="base_link" xyz="0.05 -0.14 0.1875"/>
+    <xacro:standoff_rod name="Standoff_Rod_4" parent="base_link" xyz="-0.05 0.14 0.1875"/>
+    <!-- Drive wheels -->
+    <xacro:drive_wheel side="left" name="left_wheel" parent="base_link" xyz="0 0.15 -0.0775"/>
+    <xacro:drive_wheel side="right" name="right_wheel" parent="base_link" xyz="0 -0.15 -0.0775"/>
+    <!-- Casters -->
+    <xacro:caster_wheel name="front_caster" parent="base_link" xyz="0.1 0.0 -0.0775"/>
+    <xacro:caster_wheel name="rear_caster" parent="base_link" xyz="-0.1 0.0 -0.0775"/>
+    <gazebo>
+    <plugin filename="libgazebo_ros_diff_drive.so" name="differential_drive_controller">
+        <!-- wheels -->
+        <left_joint>left_wheel_joint</left_joint>
+        <right_joint>right_wheel_joint</right_joint>
+        <!-- kinematics -->
+        <wheel_separation>0.3</wheel_separation>
+        <wheel_diameter>0.0704</wheel_diameter>
+        <!-- limits -->
+        <max_wheel_torque>1.0</max_wheel_torque>
+        <max_wheel_acceleration>2.0</max_wheel_acceleration>
+        <!-- ROS topics -->
+        <cmd_vel_topic>/cmd_vel</cmd_vel_topic>
+        <odometry_topic>/odom</odometry_topic>
+        <robot_base_frame>base_footprint</robot_base_frame>
+        <!-- output -->
+        <publish_odom>true</publish_odom>
+        <publish_odom_tf>true</publish_odom_tf>
+        <!-- update -->
+        <update_rate>50.0</update_rate>
+    </plugin>
+    </gazebo>
+    <gazebo>
+        <plugin name="barista_bot_joint_state" filename="libgazebo_ros_joint_state_publisher.so">
+        <ros>
+            <remapping>~/out:=joint_states</remapping>
+        </ros>
+        <update_rate>30</update_rate>
+        <joint_name>base_joint</joint_name>
+        <joint_name>left_wheel_joint</joint_name>
+        <joint_name>right_wheel_joint</joint_name>
+        <joint_name>front_caster_wheel_joint</joint_name>
+        <joint_name>rear_caster_wheel_joint</joint_name>
+        <joint_name>Standoff_Rod_1_Joint</joint_name>
+        <joint_name>Standoff_Rod_2_Joint</joint_name>
+        <joint_name>Standoff_Rod_3_Joint</joint_name>
+        <joint_name>Standoff_Rod_4_Joint</joint_name>
+        <joint_name>Cup_Holder_Tray_Joint</joint_name>
+        <joint_name>front_laser_joint</joint_name>
+      </plugin>
+    </gazebo>
 </robot>

File: xacro/caster_wheel.xacro (robot description, xacro)
@@ -1,51 +1,34 @@
-<?xml version="1.0"?>
-<robot xmlns:xacro="http://www.ros.org/wiki/xacro" name="barista_bot">
-<!-- FRONT CASTER WHEEL -->
-    <joint name="front_caster_wheel_joint" type="fixed">
-        <parent link="base_link"/>
-        <child link="front_caster"/>
-        <origin xyz="0.1 0.0 -0.0775" rpy="0 0 0" />
-        <axis xyz="0 0 0"/>
+<robot xmlns:xacro="http://www.ros.org/wiki/xacro">
+  <xacro:macro name="caster_wheel" params="name parent xyz">
+    <joint name="${name}_joint" type="fixed">
+      <parent link="${parent}"/>
+      <child link="${name}"/>
+      <origin xyz="${xyz}" rpy="0 0 0"/>
     </joint>
-    <link name="front_caster">
-        <visual>
-            <geometry>
-                <sphere radius="0.0352"/>
-            </geometry>
-        </visual>
-        <collision>
-            <geometry>
-                <sphere radius="0.0352"/>
-            </geometry>
-        </collision>
-        <inertial>
-            <mass value="0.5" />
-            <origin xyz="0 0 0" rpy="0 0 0" />
-            <inertia ixx="9.479166666666669e-06" ixy="0.0" ixz="0.0" iyy="9.479166666666669e-06" iyz="0.0" izz="1.5625000000000004e-05" />
-        </inertial>
+    <link name="${name}">
+      <visual>
+        <geometry>
+          <sphere radius="0.0352"/>
+        </geometry>
+      </visual>
+      <collision>
+        <geometry>
+          <sphere radius="0.0352"/>
+        </geometry>
+      </collision>
+      <inertial>
+        <mass value="0.5"/>
+        <origin xyz="0 0 0" rpy="0 0 0"/>
+        <inertia ixx="9.479e-6" ixy="0" ixz="0" iyy="9.479e-6" iyz="0" izz="1.5625e-5"/>
+      </inertial>
     </link>
-    <!-- REAR CASTER WHEEL -->
-    <joint name="rear_caster_wheel_joint" type="fixed">
-        <parent link="base_link"/>
-        <child link="back_caster"/>
-        <origin xyz="-0.1 0.0 -0.0775" rpy="0 0 0" />
-        <axis xyz="0 0 0"/>
-    </joint>
-    <link name="back_caster">
-        <visual>
-            <geometry>
-                <sphere radius="0.0352"/>
-            </geometry>
-        </visual>
-        <collision>
-            <geometry>
-                <sphere radius="0.0352"/>
-            </geometry>
-        </collision>
-        <inertial>
-            <mass value="0.5" />
-            <origin xyz="0 0 0" rpy="0 0 0" />
-            <inertia ixx="0.000247808" ixy="0.0" ixz="0.0" iyy="0.000247808" iyz="0.0" izz="0.000247808" />
-        </inertial>
-    </link>
+    <gazebo reference="${name}">
+      <mu1 value="0.0"/>
+      <mu2 value="0.0"/>
+      <kp value="10000000.0"/>
+      <kd value="100.0"/>
+      <fdir1 value="0 0 1"/>
+      <material>Gazebo/Gray</material>
+    </gazebo>
+  </xacro:macro>
 </robot>

File: xacro/cup_holder_tray.xacro (robot description, xacro)
@@ -1,29 +1,32 @@
-<?xml version="1.0"?>
-<robot xmlns:xacro="http://www.ros.org/wiki/xacro" name="barista_bot">
-    <!-- Cup_Holder_Tray_link -->
+<robot xmlns:xacro="http://www.ros.org/wiki/xacro">
+  <xacro:macro name="cup_holder_tray" params="parent">
     <joint name="Cup_Holder_Tray_Joint" type="fixed">
-        <parent link="base_link"/>
-        <child link="Cup_Holder_Tray_link"/>
-        <origin xyz="0 0 0.3425"/>
+      <parent link="${parent}"/>
+      <child link="Cup_Holder_Tray_link"/>
+      <origin xyz="0 0 0.3425"/>
     </joint>
     <link name="Cup_Holder_Tray_link">
-        <inertial>
-            <mass value="8.0" />
-            <origin xyz="0 0 0" rpy="0 0 0" />
-                <inertia ixx="0.0566" ixy="0.0" ixz="0.0" iyy="0.0566" iyz="0.0" izz="0.1024" />
-        </inertial>
-        <visual>
-            <origin xyz="0 0 0"/>
-            <geometry>
-                <cylinder radius="0.160" length="0.090"/>
-            </geometry>
-            <material name="blue"/>
-        </visual>
-        <collision>
-            <origin xyz="0 0 0"/>
-            <geometry>
-                <cylinder radius="0.160" length="0.090"/>
-            </geometry>
-        </collision>
+      <inertial>
+        <mass value="8.0"/>
+        <origin xyz="0 0 0" rpy="0 0 0"/>
+        <inertia ixx="0.0566" ixy="0" ixz="0" iyy="0.0566" iyz="0" izz="0.1024"/>
+      </inertial>
+      <visual>
+        <origin xyz="0 0 0"/>
+        <geometry>
+          <cylinder radius="0.160" length="0.090"/>
+        </geometry>
+        <material name="blue"/>
+      </visual>
+      <collision>
+        <origin xyz="0 0 0"/>
+        <geometry>
+          <cylinder radius="0.160" length="0.090"/>
+        </geometry>
+      </collision>
     </link>
+    <gazebo reference="Cup_Holder_Tray_link">
+      <material>Gazebo/Blue</material>
+    </gazebo>
+  </xacro:macro>
 </robot>

File: xacro/drive_wheel.xacro (robot description, xacro)
@@ -1,57 +1,48 @@
-<?xml version="1.0"?>
-<robot xmlns:xacro="http://www.ros.org/wiki/xacro" name="barista_bot">
-    <!-- LEFT WHEEL LINK -->
-    <joint name="left_wheel_joint" type="continuous">
-        <parent link="base_link"/>
-        <child link="left_wheel"/>
-        <origin xyz="0 0.15 -0.0775" rpy="-1.57 0 0" />
-        <axis xyz="0 0 1"/>
+<robot xmlns:xacro="http://www.ros.org/wiki/xacro">
+<xacro:macro name="drive_wheel" params="side name parent xyz">
+  <xacro:if value="${side == 'left'}">
+    <joint name="${name}_joint" type="continuous">
+      <parent link="${parent}"/>
+      <child link="${name}"/>
+      <origin xyz="${xyz}" rpy="-1.57 0 0"/>
+      <axis xyz="0 0 1"/>
     </joint>
-    <link name="left_wheel">
-        <inertial>
-            <mass value="1.5" />
-            <origin xyz="0 0 0" rpy="-1.57 0 0" />
-            <inertia ixx=" 0.000517685" ixy="0.0" ixz="0.0" iyy= "0.000517685" iyz="0.0" izz="0.00092928" />
-        </inertial>
-        <visual>
-            <origin xyz="0 0 0" rpy="0 0 0"/>
-            <geometry>
-                <cylinder radius="0.0352" length="0.0206"/>
-            </geometry>
-            <material name="black"/>
-        </visual>
-        <collision>
-            <origin xyz="0 0 0" rpy="0 0 0"/>
-            <geometry>
-                <cylinder radius="0.0352" length="0.0206"/>
-            </geometry>
-        </collision>
+  </xacro:if>
+  <xacro:unless value="${side == 'left'}">
+    <joint name="${name}_joint" type="continuous">
+      <parent link="${parent}"/>
+      <child link="${name}"/>
+      <origin xyz="${xyz}" rpy="1.57 0 0"/>
+      <axis xyz="0 0 -1"/>
+    </joint>
+  </xacro:unless>
+    <link name="${name}">
+      <inertial>
+        <mass value="1.5"/>
+        <origin xyz="0 0 0" rpy="-1.57 0 0"/>
+        <inertia ixx="0.000517685" ixy="0" ixz="0" iyy="0.000517685" iyz="0" izz="0.00092928"/>
+      </inertial>
+      <visual>
+        <origin xyz="0 0 0"/>
+        <geometry>
+          <cylinder radius="0.0352" length="0.0206"/>
+        </geometry>
+        <material name="black"/>
+      </visual>
+      <collision>
+        <origin xyz="0 0 0"/>
+        <geometry>
+          <cylinder radius="0.0352" length="0.0206"/>
+        </geometry>
+      </collision>
     </link>
-    <!-- RIGHT WHEEL LINK -->
-    <joint name="right_wheel_joint" type="continuous">
-        <parent link="base_link"/>
-        <child link="right_wheel"/>
-        <origin xyz="0 -0.15 -0.0775" rpy="1.57 0 0" />
-        <axis xyz="0 0 -1"/>
-    </joint>
-    <link name="right_wheel">
-        <inertial>
-            <mass value="1.5" />
-            <origin xyz="0 0 0" rpy="-1.575 0 0" />
-        <inertia ixx=" 0.000517685" ixy="0.0" ixz="0.0" iyy= "0.000517685" iyz="0.0" izz="0.00092928" />
-        </inertial>
-        <visual>
-            <origin xyz="0 0 0" rpy="0 0 0"/>
-            <geometry>
-                <cylinder radius="0.0352" length="0.0206"/>
-            </geometry>
-            <material name="black"/>
-        </visual>
-        <collision>
-            <origin xyz="0 0 0" rpy="0 0 0"/>
-            <geometry>
-                <cylinder radius="0.0352" length="0.0206"/>
-            </geometry>
-        </collision>
-    </link>
+    <gazebo reference="${name}">
+      <mu1 value="1.0"/>
+      <mu2 value="0.8"/>
+      <kp value="1000000.0"/>
+      <kd value="10.0"/>
+      <fdir1 value="1 0 0"/>
+      <material>Gazebo/Black</material>
+    </gazebo>
+  </xacro:macro>
 </robot>

File: xacro/laser_scanner.xacro (robot description, xacro)
@@ -1,31 +1,62 @@
-<?xml version="1.0"?>
-<robot xmlns:xacro="http://www.ros.org/wiki/xacro" name="barista_bot">
-    <!-- Laser scan -->
+<robot xmlns:xacro="http://www.ros.org/wiki/xacro">
+  <!-- <xacro:if value="${include_laser}"> -->
+  <!-- Laser Sensor -->
+  <xacro:macro name="laser_scanner" params="parent">
     <joint name="front_laser_joint" type="fixed">
-        <parent link="base_link"/>
-        <child link="front_laser"/>
-        <origin xyz="0.14 0 0.078" rpy="0 0 0" />
-        <axis xyz="0 0 0"/>
+      <parent link="${parent}"/>
+      <child link="front_laser"/>
+      <origin xyz="0.14 0.0 0.0775"/>
     </joint>
     <link name="front_laser">
-        <inertial>
-            <origin xyz="0 0 0" rpy="0 0 0" />
-            <mass value="0.05" />
-            <inertia ixx="0.000252666666667" ixy="0" ixz="0" iyy="0.000252666666667" iyz="0" izz="0.0005"/>
-        </inertial>
-        <visual>
-            <origin xyz="0 0 0" rpy="0 0 0" />
-            <geometry>
-                <mesh filename="package://barista_robot_description/meshes/sick_s3000.dae" scale="0.2 0.2 0.2"/>
-                <!-- <cylinder radius="0.025" length="0.02"/> -->
-            </geometry>
-            <material name="red"/>
-        </visual>
-        <collision>
-            <origin xyz="0 0 0" rpy="0 0 0"/>
-            <geometry>
-                <cylinder radius="0.025" length="0.02"/>
-            </geometry>
-        </collision>
+      <inertial>
+        <mass value="0.05"/>
+        <origin xyz="0 0 0"/>
+        <inertia ixx="0.000252666667" ixy="0" ixz="0" iyy="0.000252666667" iyz="0" izz="0.0005"/>
+      </inertial>
+      <visual>
+        <geometry>
+          <mesh filename="package://barista_robot_description/meshes/sick_s3000.dae" scale="0.2 0.2 0.2"/>
+        </geometry>
+        <material name="red"/>
+      </visual>
+      <collision>
+        <geometry>
+          <cylinder radius="0.025" length="0.06"/>
+        </geometry>
+      </collision>
     </link>
+    <gazebo reference="front_laser_joint">
+      <preserveFixedJoint>true</preserveFixedJoint>
+    </gazebo>
+    <gazebo reference="front_laser">
+      <material>Gazebo/DarkGrey</material>
+      <sensor name="front_laser_ray" type="ray">
+        <pose>0.03 0 0.02 0 0 0</pose>
+        <ray>
+          <scan>
+            <horizontal>
+              <samples>200</samples>
+              <resolution>1.0</resolution>
+              <min_angle>-1.57</min_angle>
+              <max_angle>1.57</max_angle>
+            </horizontal>
+          </scan>
+          <range>
+            <min>0.1</min>
+            <max>5.0</max>
+          </range>
+        </ray>
+        <always_on>true</always_on>
+        <visualize>true</visualize>
+        <update_rate>30.0</update_rate>
+        <plugin name="laser" filename="libgazebo_ros_ray_sensor.so">
+          <ros>
+            <remapping>~/out:=scan</remapping>
+          </ros>
+          <output_type>sensor_msgs/LaserScan</output_type>
+        </plugin>
+      </sensor>
+    </gazebo>
+  </xacro:macro>
+<!-- </xacro:if> -->
 </robot>

File: xacro/standoff_rod.xacro (robot description, xacro)
@@ -1,107 +1,32 @@
-<?xml version="1.0"?>
-<robot xmlns:xacro="http://www.ros.org/wiki/xacro" name="barista_bot">
-    <!-- Standoff_Rod_1_link -->
-    <joint name="Standoff_Rod_1_Joint" type="fixed">
-        <parent link="base_link"/>
-        <child link="Standoff_Rod_1_link"/>
-        <origin xyz="0.05 0.14 0.1875"/>
+<robot xmlns:xacro="http://www.ros.org/wiki/xacro">
+  <xacro:macro name="standoff_rod" params="name parent xyz">
+    <joint name="${name}_Joint" type="fixed">
+      <parent link="${parent}"/>
+      <child link="${name}_link"/>
+      <origin xyz="${xyz}"/>
     </joint>
-    <link name="Standoff_Rod_1_link">
-        <inertial>
-            <mass value="0.5" />
-            <origin xyz="0 0 0" rpy="0 0 0" />
-            <inertia ixx="0.0020291666666666665" ixy="0.0" ixz="0.0" iyy="0.0020291666666666665" iyz="0.0" izz="2.5e-05" />
-        </inertial>
-        <visual>
-            <origin xyz="0 0 0"/>
-            <geometry>
-                <cylinder radius="0.01" length="0.22"/>
-            </geometry>
-            <material name="white"/>
-        </visual>
-        <collision>
-            <origin xyz="0 0 0"/>
-            <geometry>
-                <cylinder radius="0.01" length="0.22"/>
-            </geometry>
-        </collision>
+    <link name="${name}_link">
+      <inertial>
+        <mass value="0.5"/>
+        <origin xyz="0 0 0" rpy="0 0 0"/>
+        <inertia ixx="0.0020291666666666665" ixy="0" ixz="0" iyy="0.0020291666666666665" iyz="0" izz="2.5e-05"/>
+      </inertial>
+      <visual>
+        <origin xyz="0 0 0"/>
+        <geometry>
+          <cylinder radius="0.01" length="0.22"/>
+        </geometry>
+        <material name="white"/>
+      </visual>
+      <collision>
+        <origin xyz="0 0 0"/>
+        <geometry>
+          <cylinder radius="0.01" length="0.22"/>
+        </geometry>
+      </collision>
     </link>
-    <!-- Standoff_Rod_2_link -->
-    <joint name="Standoff_Rod_2_Joint" type="fixed">
-        <parent link="base_link"/>
-        <child link="Standoff_Rod_2_link"/>
-        <origin xyz="-0.05 -0.14 0.1875"/>
-    </joint>
-    <link name="Standoff_Rod_2_link">
-        <inertial>
-            <mass value="0.5" />
-            <origin xyz="0 0 0" rpy="0 0 0" />
-            <inertia ixx="0.0020291666666666665" ixy="0.0" ixz="0.0" iyy="0.0020291666666666665" iyz="0.0" izz="2.5e-05" />
-        </inertial>
-        <visual>
-            <origin xyz="0 0 0"/>
-            <geometry>
-                <cylinder radius="0.01" length="0.22"/>
-            </geometry>
-            <material name="white"/>
-        </visual>
-        <collision>
-            <origin xyz="0 0 0"/>
-            <geometry>
-                <cylinder radius="0.01" length="0.22"/>
-            </geometry>
-        </collision>
-    </link>
-    <!-- Standoff_Rod_3_link -->
-    <joint name="Standoff_Rod_3_Joint" type="fixed">
-        <parent link="base_link"/>
-        <child link="Standoff_Rod_3_link"/>
-        <origin xyz="0.05 -0.14 0.1875"/>
-    </joint>
-    <link name="Standoff_Rod_3_link">
-        <inertial>
-            <mass value="0.5" />
-            <origin xyz="0 0 0" rpy="0 0 0" />
-            <inertia ixx="0.0020291666666666665" ixy="0.0" ixz="0.0" iyy="0.0020291666666666665" iyz="0.0" izz="2.5e-05" />
-        </inertial>
-        <visual>
-            <origin xyz="0 0 0"/>
-            <geometry>
-                <cylinder radius="0.01" length="0.22"/>
-            </geometry>
-            <material name="white"/>
-        </visual>
-        <collision>
-            <origin xyz="0 0 0"/>
-            <geometry>
-                <cylinder radius="0.01" length="0.22"/>
-            </geometry>
-        </collision>
-    </link>
-    <!-- Standoff_Rod_4_link -->
-    <joint name="Standoff_Rod_4_Joint" type="fixed">
-        <parent link="base_link"/>
-        <child link="Standoff_Rod_4_link"/>
-        <origin xyz="-0.05 0.14 0.1875"/>
-    </joint>
-    <link name="Standoff_Rod_4_link">
-        <inertial>
-            <mass value="0.5" />
-            <origin xyz="0 0 0" rpy="0 0 0" />
-            <inertia ixx="0.0020291666666666665" ixy="0.0" ixz="0.0" iyy="0.0020291666666666665" iyz="0.0" izz="2.5e-05" />
-        </inertial>
-        <visual>
-            <origin xyz="0 0 0"/>
-            <geometry>
-                <cylinder radius="0.01" length="0.22"/>
-            </geometry>
-            <material name="white"/>
-        </visual>
-        <collision>
-            <origin xyz="0 0 0"/>
-            <geometry>
-                <cylinder radius="0.01" length="0.22"/>
-            </geometry>
-        </collision>
-    </link>
+    <gazebo reference="${name}_link">
+      <material>Gazebo/white</material>
+    </gazebo>
+  </xacro:macro>
 </robot>
