Commit message: corrected added include laser if xacro

File: xacro/barista_robot_model.urdf.xacro (robot description, xacro)
@@ -1,9 +1,4 @@
 <?xml version="1.0"?>
 <robot xmlns:xacro="http://www.ros.org/wiki/xacro" name="barista_bot">
-    <!-- Conditional laser -->
-    <!-- <xacro:arg name="include_laser" default="true"/> -->
-    <!-- <xacro:if value="$(arg include_laser)"> -->
-        <!-- <xacro:laser_scanner parent="base_link"/> -->
-    <!-- </xacro:if> -->
     <!-- Arguments -->
     <xacro:arg name="robot_name" default="barista_bot"/>
@@ -57,6 +52,9 @@
     <xacro:caster_wheel name="front_caster" parent="base_link" xyz="0.1 0.0 -0.0775"/>
     <xacro:caster_wheel name="rear_caster" parent="base_link" xyz="-0.1 0.0 -0.0775"/>
+    <!-- Laser include -->
+    <xacro:laser_scanner include_laser="True"/>
     <!-- Laser -->
-    <xacro:laser_scanner parent="base_link"/>
+    <!-- <xacro:macro name="laser_scanner" params="include_laser:=true"> -->
+    <!-- <xacro:laser_scanner parent="base_link"/> -->
     <gazebo>
     <plugin filename="libgazebo_ros_diff_drive.so" name="differential_drive_controller">

File: xacro/laser_scanner.xacro (robot description, xacro)
@@ -1,6 +1,7 @@
 <robot xmlns:xacro="http://www.ros.org/wiki/xacro">
-  <xacro:macro name="laser_scanner" params="parent">
+  <xacro:macro name="laser_scanner" params="include_laser:=true">
+    <xacro:if value="${include_laser}">
     <joint name="front_laser_joint" type="fixed">
-      <parent link="${parent}"/>
+      <parent link="base_link"/>
       <child link="front_laser"/>
       <origin xyz="0.14 0.0 0.0775"/>
@@ -56,4 +57,5 @@
       </sensor>
     </gazebo>
+   </xacro:if>
   </xacro:macro>
 </robot>

Commit message: update with solutions, remove join state publisher for static joint LOL

File: xacro/barista_robot_model.urdf.xacro (robot description, xacro)
@@ -85,15 +85,15 @@
         </ros>
         <update_rate>30</update_rate>
-        <joint_name>base_joint</joint_name>
+        <!-- <joint_name>base_joint</joint_name> -->
         <joint_name>left_wheel_joint</joint_name>
         <joint_name>right_wheel_joint</joint_name>
-        <joint_name>front_caster_wheel_joint</joint_name>
+        <!-- <joint_name>front_caster_wheel_joint</joint_name>
         <joint_name>rear_caster_wheel_joint</joint_name>
-        <joint_name>Standoff_Rod_1_Joint</joint_name>
-        <joint_name>Standoff_Rod_2_Joint</joint_name>
-        <joint_name>Standoff_Rod_3_Joint</joint_name>
-        <joint_name>Standoff_Rod_4_Joint</joint_name>
-        <joint_name>Cup_Holder_Tray_Joint</joint_name>
-        <joint_name>front_laser_joint</joint_name>
+        <joint_name>Standoff_Rod_1_joint</joint_name>
+        <joint_name>Standoff_Rod_2_joint</joint_name>
+        <joint_name>Standoff_Rod_3_joint</joint_name>
+        <joint_name>Standoff_Rod_4_joint</joint_name>
+        <joint_name>Cup_Holder_Tray_joint</joint_name>
+        <joint_name>front_laser_joint</joint_name> -->
       </plugin>
     </gazebo>

File: xacro/cup_holder_tray.xacro (robot description, xacro)
@@ -1,5 +1,5 @@
 <robot xmlns:xacro="http://www.ros.org/wiki/xacro">
   <xacro:macro name="cup_holder_tray" params="parent">
-    <joint name="Cup_Holder_Tray_Joint" type="fixed">
+    <joint name="Cup_Holder_Tray_joint" type="fixed">
       <parent link="${parent}"/>
       <child link="Cup_Holder_Tray_link"/>

File: xacro/laser_scanner.xacro (robot description, xacro)
@@ -37,6 +37,6 @@
               <samples>200</samples>
               <resolution>1.0</resolution>
-              <min_angle>-1.57</min_angle>
-              <max_angle>1.57</max_angle>
+              <min_angle>-3.14</min_angle>
+              <max_angle>3.147</max_angle>
             </horizontal>
           </scan>

File: xacro/standoff_rod.xacro (robot description, xacro)
@@ -1,5 +1,5 @@
 <robot xmlns:xacro="http://www.ros.org/wiki/xacro">
   <xacro:macro name="standoff_rod" params="name parent xyz">
-    <joint name="${name}_Joint" type="fixed">
+    <joint name="${name}_joint" type="fixed">
       <parent link="${parent}"/>
       <child link="${name}_link"/>
